File: AddrLatch.sch (KiCad schematic (older format))
At the start: 6 parts, among them U14 74LVC574AD, U15 74LVC574AD, U16 74LVC574AD

Commit message: Export gerbers just to test
Parts:
- C19, C20, C21: LCSC Part (none) -> C15850
- U14, U15, U16: LCSC Part (none) -> C6097
Changed lines of the file:
@@
 F 2 "stdpads:SOIC-20W_7.5mm" H 4400 2550 50  0001 C TNN
 F 3 "" H 4400 3300 60  0001 C CNN
+F 4 "C6097" H 4400 3200 50  0001 C CNN "LCSC Part"
 	1    4400 3200
 	1    0    0    -1
@@
 F 2 "stdpads:SOIC-20W_7.5mm" H 4400 1350 50  0001 C TNN
 F 3 "" H 4400 2100 60  0001 C CNN
+F 4 "C6097" H 4400 2000 50  0001 C CNN "LCSC Part"
 	1    4400 2000
 	1    0    0    -1
@@
 F 2 "stdpads:SOIC-20W_7.5mm" H 4400 3750 50  0001 C TNN
 F 3 "" H 4400 4500 60  0001 C CNN
+F 4 "C6097" H 4400 4400 50  0001 C CNN "LCSC Part"
 	1    4400 4400
 	1    0    0    -1
@@
 F 2 "stdpads:C_0805" H 6900 3200 50  0001 C CNN
 F 3 "~" H 6900 3200 50  0001 C CNN
+F 4 "C15850" H 6900 3200 50  0001 C CNN "LCSC Part"
 	1    6900 3200
 	-1   0    0    -1
@@
 F 2 "stdpads:C_0805" H 6500 3200 50  0001 C CNN
 F 3 "~" H 6500 3200 50  0001 C CNN
+F 4 "C15850" H 6500 3200 50  0001 C CNN "LCSC Part"
 	1    6500 3200
 	-1   0    0    -1
@@
 F 2 "stdpads:C_0805" H 6100 3200 50  0001 C CNN
 F 3 "~" H 6100 3200 50  0001 C CNN
+F 4 "C15850" H 6100 3200 50  0001 C CNN "LCSC Part"
 	1    6100 3200
 	-1   0    0    -1
