File: BusControl.sch (KiCad schematic (older format))
At the start: 29 parts, among them U17 74LVC74AD, U18 74LVC74AD, U19 74LVC74AD, U20 74LVC86AD, U21 74LVC32AD, U22 74LVC02AD, U23 74LVC00AD, U24 74LVC125AD, U25 74LVC32AD, U26 74LVC125AD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

Commit message: Export gerbers just to test
Parts:
- C10, C11, C12, C13, C14, C15, C36, C46, C6, C7, C8, C9: LCSC Part (none) -> C15850
- R11, R8: LCSC Part C25190 -> C17408
- U17, U18, U19, U35, U36, U37: LCSC Part (none) -> C7864
- U20: LCSC Part (none) -> C548853
- U21, U25, U34, U42: LCSC Part (none) -> C7852
- U22: LCSC Part (none) -> C7804
- U23: LCSC Part (none) -> C7802
- U24, U26: LCSC Part (none) -> C7661
