File: CtrlStatReg.sch (KiCad schematic (older format))
At the start: 13 parts, among them Q5 MMBT3904, U18 74LVC74AD, U19 74LVC74AD, U22 74LVC02AD, U24 74LVC125AD, U35 74LVC74AD, U36 74LVC74AD, U37 74LVC74AD

Commit message: Export gerbers just to test
Parts:
- C43, C44, C45: LCSC Part (none) -> C15850
- R31, R32: LCSC Part C25190 -> C17513
- U18, U19, U35, U36, U37: LCSC Part (none) -> C7864
- U22: LCSC Part (none) -> C7804
- U24: LCSC Part (none) -> C7661
Changed lines of the file:
@@
 F 2 "stdpads:C_0805" H 9150 5100 50  0001 C CNN
 F 3 "~" H 9150 5100 50  0001 C CNN
+F 4 "C15850" H 9150 5100 50  0001 C CNN "LCSC Part"
 	1    9150 5100
 	-1   0    0    -1
@@
 F 2 "stdpads:C_0805" H 9550 5100 50  0001 C CNN
 F 3 "~" H 9550 5100 50  0001 C CNN
+F 4 "C15850" H 9550 5100 50  0001 C CNN "LCSC Part"
 	1    9550 5100
 	-1   0    0    -1
@@
 F 2 "stdpads:C_0805" H 9950 5100 50  0001 C CNN
 F 3 "~" H 9950 5100 50  0001 C CNN
+F 4 "C15850" H 9950 5100 50  0001 C CNN "LCSC Part"
 	1    9950 5100
 	-1   0    0    -1
@@
 F 2 "stdpads:SOIC-14_3.9mm" H 10550 1500 50  0001 C CNN
 F 3 "74xx/74hc_hct74.pdf" H 10550 1500 50  0001 C CNN
+F 4 "C7864" H 10550 1500 50  0001 C CNN "LCSC Part"
 	2    10550 1500
 	1    0    0    -1
@@
 F 2 "stdpads:SOIC-14_3.9mm" H 3250 6750 50  0001 C CNN
 F 3 "74xx/74hc_hct74.pdf" H 3250 6750 50  0001 C CNN
+F 4 "C7864" H 3250 6750 50  0001 C CNN "LCSC Part"
 	2    3250 6750
 	1    0    0    -1
@@
 F 2 "stdpads:SOIC-14_3.9mm" H 3250 5850 50  0001 C CNN
 F 3 "74xx/74hc_hct74.pdf" H 3250 5850 50  0001 C CNN
+F 4 "C7864" H 3250 5850 50  0001 C CNN "LCSC Part"
 	1    3250 5850
 	1    0    0    -1
@@
 F 2 "stdpads:R_0805" H 5550 6250 50  0001 C CNN
 F 3 "~" H 5550 6250 50  0001 C CNN
-F 4 "C25190" H 5550 6250 50  0001 C CNN "LCSC Part"
+F 4 "C17513" H 5550 6250 50  0001 C CNN "LCSC Part"
 	1    5550 6250
 	0    1    1    0
@@
 F 2 "stdpads:SOIC-14_3.9mm" H 5150 6650 50  0001 C CNN
 F 3 "http://www.ti.com/lit/gpn/sn74LS02" H 5150 6650 50  0001 C CNN
+F 4 "C7804" H 5150 6650 50  0001 C CNN "LCSC Part"
 	3    5150 6650
 	1    0    0    -1
@@
 F 2 "stdpads:R_0805" H 5550 6650 50  0001 C CNN
 F 3 "~" H 5550 6650 50  0001 C CNN
-F 4 "C25190" H 5550 6650 50  0001 C CNN "LCSC Part"
+F 4 "C17513" H 5550 6650 50  0001 C CNN "LCSC Part"
 	1    5550 6650
 	0    1    1    0
@@
 F 2 "stdpads:SOIC-14_3.9mm" H 3250 1350 50  0001 C CNN
 F 3 "74xx/74hc_hct74.pdf" H 3250 1350 50  0001 C CNN
+F 4 "C7864" H 3250 1350 50  0001 C CNN "LCSC Part"
 	1    3250 1350
 	1    0    0    -1
@@
 F 2 "stdpads:SOIC-14_3.9mm" H 3250 4050 50  0001 C CNN
 F 3 "74xx/74hc_hct74.pdf" H 3250 4050 50  0001 C CNN
+F 4 "C7864" H 3250 4050 50  0001 C CNN "LCSC Part"
 	2    3250 4050
 	1    0    0    -1
@@
 F 2 "stdpads:SOIC-14_3.9mm" H 3250 2250 50  0001 C CNN
 F 3 "74xx/74hc_hct74.pdf" H 3250 2250 50  0001 C CNN
+F 4 "C7864" H 3250 2250 50  0001 C CNN "LCSC Part"
 	1    3250 2250
 	1    0    0    -1
@@
 F 2 "stdpads:SOIC-14_3.9mm" H 3250 3150 50  0001 C CNN
 F 3 "74xx/74hc_hct74.pdf" H 3250 3150 50  0001 C CNN
+F 4 "C7864" H 3250 3150 50  0001 C CNN "LCSC Part"
 	1    3250 3150
 	1    0    0    -1
@@
 F 2 "stdpads:SOIC-14_3.9mm" H 3250 4950 50  0001 C CNN
 F 3 "74xx/74hc_hct74.pdf" H 3250 4950 50  0001 C CNN
+F 4 "C7864" H 3250 4950 50  0001 C CNN "LCSC Part"
 	2    3250 4950
 	1    0    0    -1
@@
 F 2 "stdpads:SOIC-14_3.9mm" H 5150 6250 50  0001 C CNN
 F 3 "http://www.ti.com/lit/gpn/sn74LS02" H 5150 6250 50  0001 C CNN
+F 4 "C7804" H 5150 6250 50  0001 C CNN "LCSC Part"
 	4    5150 6250
 	1    0    0    -1
@@
 F 2 "stdpads:SOIC-14_3.9mm" H 4150 4850 50  0001 C CNN
 F 3 "http://www.ti.com/lit/gpn/sn74LS125" H 4150 4850 50  0001 C CNN
+F 4 "C7661" H 4150 4850 50  0001 C CNN "LCSC Part"
 	3    4150 4850
 	1    0    0    -1
@@
 F 2 "stdpads:SOIC-14_3.9mm" H 4150 3050 50  0001 C CNN
 F 3 "http://www.ti.com/lit/gpn/sn74LS125" H 4150 3050 50  0001 C CNN
+F 4 "C7661" H 4150 3050 50  0001 C CNN "LCSC Part"
 	4    4150 3050
 	1    0    0    -1
