File: DataReg.sch (KiCad schematic (older format))
At the start: 39 parts, among them U10 74LVC574AD, U11 74LVC574AD, U12 74LVC574AD, U13 74LVC574AD, U29 74LVC574AD, U30 74LVC574AD, U31 74LVC574AD, U32 74LVC574AD, U33 74LVC574AD, U35 74LVC74AD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

Commit message: Export gerbers just to test
Parts:
- C22, C23, C24, C25, C26, C27, C28, C29, C30, C38, C39, C40, C41, C42, C47, C48, C49, C50: LCSC Part (none) -> C15850
- R9: LCSC Part C25190 -> C17561
- U10, U11, U12, U13, U29, U30, U31, U32, U33, U38, U39, U40, U41, U5, U6, U7, U8, U9: LCSC Part (none) -> C6097
- U35: LCSC Part (none) -> C7864
- U42: LCSC Part (none) -> C7852
Changed lines of the file:
@@
 F 2 "stdpads:C_0805" H 9300 5850 50  0001 C CNN
 F 3 "~" H 9300 5850 50  0001 C CNN
+F 4 "C15850" H 9300 5850 50  0001 C CNN "LCSC Part"
 	1    9300 5850
 	-1   0    0    -1
@@
 F 2 "stdpads:C_0805" H 10100 5850 50  0001 C CNN
 F 3 "~" H 10100 5850 50  0001 C CNN
+F 4 "C15850" H 10100 5850 50  0001 C CNN "LCSC Part"
 	1    10100 5850
 	-1   0    0    -1
@@
 F 2 "stdpads:C_0805" H 9700 5850 50  0001 C CNN
 F 3 "~" H 9700 5850 50  0001 C CNN
+F 4 "C15850" H 9700 5850 50  0001 C CNN "LCSC Part"
 	1    9700 5850
 	-1   0    0    -1
@@
 F 2 "stdpads:C_0805" H 10500 5850 50  0001 C CNN
 F 3 "~" H 10500 5850 50  0001 C CNN
+F 4 "C15850" H 10500 5850 50  0001 C CNN "LCSC Part"
 	1    10500 5850
 	-1   0    0    -1
@@
 F 2 "stdpads:C_0805" H 10100 5450 50  0001 C CNN
 F 3 "~" H 10100 5450 50  0001 C CNN
+F 4 "C15850" H 10100 5450 50  0001 C CNN "LCSC Part"
 	1    10100 5450
 	-1   0    0    -1
@@
 F 2 "stdpads:C_0805" H 9700 5450 50  0001 C CNN
 F 3 "~" H 9700 5450 50  0001 C CNN
+F 4 "C15850" H 9700 5450 50  0001 C CNN "LCSC Part"
 	1    9700 5450
 	-1   0    0    -1
@@
 F 2 "stdpads:C_0805" H 10500 5450 50  0001 C CNN
 F 3 "~" H 10500 5450 50  0001 C CNN
+F 4 "C15850" H 10500 5450 50  0001 C CNN "LCSC Part"
 	1    10500 5450
 	-1   0    0    -1
@@
 F 2 "stdpads:C_0805" H 10900 5450 50  0001 C CNN
 F 3 "~" H 10900 5450 50  0001 C CNN
+F 4 "C15850" H 10900 5450 50  0001 C CNN "LCSC Part"
 	1    10900 5450
 	-1   0    0    -1
@@
 F 2 "stdpads:C_0805" H 9300 5450 50  0001 C CNN
 F 3 "~" H 9300 5450 50  0001 C CNN
+F 4 "C15850" H 9300 5450 50  0001 C CNN "LCSC Part"
 	1    9300 5450
 	-1   0    0    -1
@@
 F 2 "stdpads:SOIC-20W_7.5mm" H 2300 4700 50  0001 C TNN
 F 3 "" H 2300 5450 60  0001 C CNN
+F 4 "C6097" H 2300 5350 50  0001 C CNN "LCSC Part"
 	1    2300 5350
 	1    0    0    -1
@@
 F 2 "stdpads:SOIC-20W_7.5mm" H 2300 3500 50  0001 C TNN
 F 3 "" H 2300 4250 60  0001 C CNN
+F 4 "C6097" H 2300 4150 50  0001 C CNN "LCSC Part"
 	1    2300 4150
 	1    0    0    -1
@@
 F 2 "stdpads:SOIC-20W_7.5mm" H 2300 2300 50  0001 C TNN
 F 3 "" H 2300 3050 60  0001 C CNN
+F 4 "C6097" H 2300 2950 50  0001 C CNN "LCSC Part"
 	1    2300 2950
 	1    0    0    -1
@@
 F 2 "stdpads:SOIC-20W_7.5mm" H 2300 1100 50  0001 C TNN
 F 3 "" H 2300 1850 60  0001 C CNN
+F 4 "C6097" H 2300 1750 50  0001 C CNN "LCSC Part"
 	1    2300 1750
 	1    0    0    -1
@@
 F 2 "stdpads:SOIC-20W_7.5mm" H 2300 5900 50  0001 C TNN
 F 3 "" H 2300 6650 60  0001 C CNN
+F 4 "C6097" H 2300 6550 50  0001 C CNN "LCSC Part"
 	1    2300 6550
 	1    0    0    -1
@@
 F 2 "stdpads:SOIC-20W_7.5mm" H 3600 5900 50  0001 C TNN
 F 3 "" H 3600 6650 60  0001 C CNN
+F 4 "C6097" H 3600 6550 50  0001 C CNN "LCSC Part"
 	1    3600 6550
 	1    0    0    -1
@@
 F 2 "stdpads:SOIC-14_3.9mm" H 8800 1700 50  0001 C CNN
 F 3 "http://www.ti.com/lit/gpn/sn74LS32" H 8800 1700 50  0001 C CNN
+F 4 "C7852" H 8800 1700 50  0001 C CNN "LCSC Part"
 	3    8800 1700
 	-1   0    0    -1
@@
 F 2 "stdpads:SOIC-20W_7.5mm" H 3600 4700 50  0001 C TNN
 F 3 "" H 3600 5450 60  0001 C CNN
+F 4 "C6097" H 3600 5350 50  0001 C CNN "LCSC Part"
 	1    3600 5350
 	1    0    0    -1
@@
 F 2 "stdpads:SOIC-20W_7.5mm" H 3600 3500 50  0001 C TNN
 F 3 "" H 3600 4250 60  0001 C CNN
+F 4 "C6097" H 3600 4150 50  0001 C CNN "LCSC Part"
 	1    3600 4150
 	1    0    0    -1
@@
 F 2 "stdpads:SOIC-20W_7.5mm" H 3600 2300 50  0001 C TNN
 F 3 "" H 3600 3050 60  0001 C CNN
+F 4 "C6097" H 3600 2950 50  0001 C CNN "LCSC Part"
 	1    3600 2950
 	1    0    0    -1
@@
 F 2 "stdpads:SOIC-20W_7.5mm" H 3600 1100 50  0001 C TNN
 F 3 "" H 3600 1850 60  0001 C CNN
+F 4 "C6097" H 3600 1750 50  0001 C CNN "LCSC Part"
 	1    3600 1750
 	1    0    0    -1
@@
 F 2 "stdpads:C_0805" H 10100 5050 50  0001 C CNN
 F 3 "~" H 10100 5050 50  0001 C CNN
+F 4 "C15850" H 10100 5050 50  0001 C CNN "LCSC Part"
 	1    10100 5050
 	-1   0    0    -1
@@
 F 2 "stdpads:C_0805" H 9700 5050 50  0001 C CNN
 F 3 "~" H 9700 5050 50  0001 C CNN
+F 4 "C15850" H 9700 5050 50  0001 C CNN "LCSC Part"
 	1    9700 5050
 	-1   0    0    -1
@@
 F 2 "stdpads:C_0805" H 10500 5050 50  0001 C CNN
 F 3 "~" H 10500 5050 50  0001 C CNN
+F 4 "C15850" H 10500 5050 50  0001 C CNN "LCSC Part"
 	1    10500 5050
 	-1   0    0    -1
@@
 F 2 "stdpads:C_0805" H 10900 5050 50  0001 C CNN
 F 3 "~" H 10900 5050 50  0001 C CNN
+F 4 "C15850" H 10900 5050 50  0001 C CNN "LCSC Part"
 	1    10900 5050
 	-1   0    0    -1
@@
 F 2 "stdpads:C_0805" H 9300 5050 50  0001 C CNN
 F 3 "~" H 9300 5050 50  0001 C CNN
+F 4 "C15850" H 9300 5050 50  0001 C CNN "LCSC Part"
 	1    9300 5050
 	-1   0    0    -1
@@
 F 2 "stdpads:R_0805" H 4300 4600 50  0001 C CNN
 F 3 "~" H 4300 4600 50  0001 C CNN
-F 4 "C25190" H 4300 4600 50  0001 C CNN "LCSC Part"
+F 4 "C17561" H 4300 4600 50  0001 C CNN "LCSC Part"
 	1    4300 4600
 	0    -1   1    0
@@
 F 2 "stdpads:SOIC-20W_7.5mm" H 7900 1400 50  0001 C TNN
 F 3 "" H 7900 2150 60  0001 C CNN
+F 4 "C6097" H 7900 2050 50  0001 C CNN "LCSC Part"
 	1    7900 2050
 	-1   0    0    -1
@@
 F 2 "stdpads:SOIC-20W_7.5mm" H 7900 2600 50  0001 C TNN
 F 3 "" H 7900 3350 60  0001 C CNN
+F 4 "C6097" H 7900 3250 50  0001 C CNN "LCSC Part"
 	1    7900 3250
 	-1   0    0    -1
@@
 F 2 "stdpads:SOIC-20W_7.5mm" H 7900 3800 50  0001 C TNN
 F 3 "" H 7900 4550 60  0001 C CNN
+F 4 "C6097" H 7900 4450 50  0001 C CNN "LCSC Part"
 	1    7900 4450
 	-1   0    0    -1
@@
 F 2 "stdpads:SOIC-20W_7.5mm" H 7900 5000 50  0001 C TNN
 F 3 "" H 7900 5750 60  0001 C CNN
+F 4 "C6097" H 7900 5650 50  0001 C CNN "LCSC Part"
 	1    7900 5650
 	-1   0    0    -1
@@
 F 2 "stdpads:SOIC-20W_7.5mm" H 6700 1400 50  0001 C TNN
 F 3 "" H 6700 2150 60  0001 C CNN
+F 4 "C6097" H 6700 2050 50  0001 C CNN "LCSC Part"
 	1    6700 2050
 	-1   0    0    -1
@@
 F 2 "stdpads:SOIC-20W_7.5mm" H 6700 2600 50  0001 C TNN
 F 3 "" H 6700 3350 60  0001 C CNN
+F 4 "C6097" H 6700 3250 50  0001 C CNN "LCSC Part"
 	1    6700 3250
 	-1   0    0    -1
@@
 F 2 "stdpads:SOIC-20W_7.5mm" H 6700 3800 50  0001 C TNN
 F 3 "" H 6700 4550 60  0001 C CNN
+F 4 "C6097" H 6700 4450 50  0001 C CNN "LCSC Part"
 	1    6700 4450
 	-1   0    0    -1
@@
 F 2 "stdpads:SOIC-20W_7.5mm" H 6700 5000 50  0001 C TNN
 F 3 "" H 6700 5750 60  0001 C CNN
+F 4 "C6097" H 6700 5650 50  0001 C CNN "LCSC Part"
 	1    6700 5650
 	-1   0    0    -1
@@
 F 2 "stdpads:C_0805" H 9300 6250 50  0001 C CNN
 F 3 "~" H 9300 6250 50  0001 C CNN
+F 4 "C15850" H 9300 6250 50  0001 C CNN "LCSC Part"
 	1    9300 6250
 	-1   0    0    -1
@@
 F 2 "stdpads:C_0805" H 10100 6250 50  0001 C CNN
 F 3 "~" H 10100 6250 50  0001 C CNN
+F 4 "C15850" H 10100 6250 50  0001 C CNN "LCSC Part"
 	1    10100 6250
 	-1   0    0    -1
@@
 F 2 "stdpads:C_0805" H 9700 6250 50  0001 C CNN
 F 3 "~" H 9700 6250 50  0001 C CNN
+F 4 "C15850" H 9700 6250 50  0001 C CNN "LCSC Part"
 	1    9700 6250
 	-1   0    0    -1
@@
 F 2 "stdpads:C_0805" H 10500 6250 50  0001 C CNN
 F 3 "~" H 10500 6250 50  0001 C CNN
+F 4 "C15850" H 10500 6250 50  0001 C CNN "LCSC Part"
 	1    10500 6250
 	-1   0    0    -1
@@
 F 2 "stdpads:SOIC-14_3.9mm" H 4800 7000 50  0001 C CNN
 F 3 "74xx/74hc_hct74.pdf" H 4800 7000 50  0001 C CNN
+F 4 "C7864" H 4800 7000 50  0001 C CNN "LCSC Part"
 	2    4800 7000
 	1    0    0    -1
@@
 F 2 "stdpads:SOIC-14_3.9mm" H 4700 4600 50  0001 C CNN
 F 3 "http://www.ti.com/lit/gpn/sn74LS32" H 4700 4600 50  0001 C CNN
+F 4 "C7852" H 4700 4600 50  0001 C CNN "LCSC Part"
 	2    4700 4600
 	-1   0    0    -1
@@
 F 2 "stdpads:SOIC-14_3.9mm" H 8800 1300 50  0001 C CNN
 F 3 "http://www.ti.com/lit/gpn/sn74LS32" H 8800 1300 50  0001 C CNN
+F 4 "C7852" H 8800 1300 50  0001 C CNN "LCSC Part"
 	1    8800 1300
 	-1   0    0    -1
