File: ESP32.sch (KiCad schematic (older format))
At the start: 36 parts, among them J4 JTAG, Q1 MMBT3904, Q2 MMBT3904, Q3 MMBT3904, Q4 MMBT3904, U1 ESP-WROVER-32, U3 CH340G, Y1 12M

Commit message: Export gerbers just to test
Parts:
- added R34, R35, R36: 10k, stdpads:R_0805, symbol Device:R_Small
- C1, C2: LCSC Part C1653 -> C1804
- C3: LCSC Part (none) -> C28233
- C31, C32, C33, C37: LCSC Part (none) -> C15850
- J4: LCSC Part (none) -> C5665
- R10: LCSC Part C25190 -> C17513
- R12, R15: LCSC Part C25190 -> C17408
- R13, R14, R16: LCSC Part C31850 -> C17414
- R17, R19, R27: LCSC Part C21190 -> C17513
- R22: value 1k -> 10k; LCSC Part C25190 -> C17414
- R25, R26, R33: LCSC Part C25190 -> C17561
- R28: LCSC Part (none) -> C17414
- R29, R30: LCSC Part C25804 -> C17414
- U1: LCSC Part (none) -> C967023
Connections:
- net +3V3: now also R34.1, R35.1
- net GND: now also R36.2
- net N~CS~: now also R35.2
- net RDCLK: now also R36.1
- net WRCLK: now also R34.2
- net ~EN~: now also R22.1; no longer R22.2
- net at Q3.1 (B): now also R22.2; no longer R22.1
Other:
- note added: "IO0: pull-up disables ESP32 serial download\nIO2: pull-down disables ESP32 test mode\nIO13 (TCK): pull-down prevents JTAG TCK clock pulse at power-on\nIO14 (TMS): pull-up causes JTAG to reset state if accidental TCK pulse\nIO15 (TDO): pull up for debug output, down for fast/quiet boot (internal pull-up)\nIO12 (TDI): pull up for 1.8V flash, down for 3.3V flash (internal pull-down)"
- note added: "internal pulldown on IO12"
- note added: "internal pulldown on IO13"
- note added: "internal pulldown on IO2"
- note added: "internal pulldown on IO4"
- note added: "internal pullup on IO0, toggles at boot"
- note added: "internal pullup on IO14, toggles at boot"
- note added: "internal pullup on IO15, toggles at boot"
- note added: "internal pullup on IO5, toggles at boot"
- note removed: "IO0: pull-up disables ESP32 serial download\nIO2: pull-down disables ESP32 test mode\nTCK: pull-down prevents JTAG TCK clock pulse at power-on\nTMS: pull-up causes JTAG to reset state if accidental TCK pulse\nTDO: pull up for debug output, down for fast/quiet boot (internal pull-up)\nTDI: pull up for 1.8V flash, down for 3.3V flash (internal pull-down)"
- note removed: "internal weak pulldown on IO12"
- note removed: "internal weak pulldown on IO13"
- note removed: "internal weak pulldown on IO2"
- note removed: "internal weak pulldown on IO4"
- note removed: "internal weak pullup on IO0"
- note removed: "internal weak pullup on IO14"
- note removed: "internal weak pullup on IO15"
- note removed: "internal weak pullup on IO5"
Changed lines of the file:
@@
 F 2 "stdpads:ESP32-WROVER_WROOM-32_WROVER" H 5650 600 50  0001 C CNN
 F 3 "" H 5200 2400 60  0001 C CNN
+F 4 "C967023" H 5650 1950 50  0001 C CNN "LCSC Part"
 	1    5650 1950
 	1    0    0    -1
@@
 F 2 "stdpads:R_0805" H 2500 4700 50  0001 C CNN
 F 3 "~" H 2500 4700 50  0001 C CNN
-F 4 "C21190" H 2500 4700 50  0001 C CNN "LCSC Part"
+F 4 "C17513" H 2500 4700 50  0001 C CNN "LCSC Part"
 	1    2500 4700
 	-1   0    0    -1
@@
 F 2 "stdpads:C_0805" H 2600 5400 50  0001 C CNN
 F 3 "~" H 2600 5400 50  0001 C CNN
-F 4 "C1653" H 2600 5400 50  0001 C CNN "LCSC Part"
+F 4 "C1804" H 2600 5400 50  0001 C CNN "LCSC Part"
 	1    2600 5400
 	-1   0    0    -1
@@
 F 2 "stdpads:R_0805" H 4850 4900 50  0001 C CNN
 F 3 "~" H 4850 4900 50  0001 C CNN
-F 4 "C25804" H 4850 4900 50  0001 C CNN "LCSC Part"
+F 4 "C17414" H 4850 4900 50  0001 C CNN "LCSC Part"
 	1    4850 4900
 	0    -1   1    0
@@
 F 2 "stdpads:R_0805" H 4850 4400 50  0001 C CNN
 F 3 "~" H 4850 4400 50  0001 C CNN
-F 4 "C25804" H 4850 4400 50  0001 C CNN "LCSC Part"
+F 4 "C17414" H 4850 4400 50  0001 C CNN "LCSC Part"
 	1    4850 4400
 	0    -1   1    0
@@
 F 2 "stdpads:C_0805" H 2200 5400 50  0001 C CNN
 F 3 "~" H 2200 5400 50  0001 C CNN
-F 4 "C1653" H 2200 5400 50  0001 C CNN "LCSC Part"
+F 4 "C1804" H 2200 5400 50  0001 C CNN "LCSC Part"
 	1    2200 5400
 	-1   0    0    -1
@@
 F 2 "stdpads:R_0805" H 2150 2450 50  0001 C CNN
 F 3 "~" H 2150 2450 50  0001 C CNN
-F 4 "C25190" H 2150 2450 50  0001 C CNN "LCSC Part"
+F 4 "C17408" H 2150 2450 50  0001 C CNN "LCSC Part"
 	1    2150 2450
 	0    -1   1    0
@@
 F 2 "Connector_IDC:IDC-Header_2x05_P2.54mm_Vertical" H 1550 2650 50  0001 C CNN
 F 3 "~" H 1550 2650 50  0001 C CNN
+F 4 "C5665" H 1550 2650 50  0001 C CNN "LCSC Part"
 	1    1550 2650
 	1    0    0    -1
@@
 $EndComp
 Text Notes 3000 7100 0    50   ~ 0
-IO0: pull-up disables ESP32 serial download\nIO2: pull-down disables ESP32 test mode\nTCK: pull-down prevents JTAG TCK clock pulse at power-on\nTMS: pull-up causes JTAG to reset state if accidental TCK pulse\nTDO: pull up for debug output, down for fast/quiet boot (internal pull-up)\nTDI:  pull up for 1.8V flash, down for 3.3V flash (internal pull-down)
+IO0:         pull-up disables ESP32 serial download\nIO2:         pull-down disables ESP32 test mode\nIO13 (TCK): pull-down prevents JTAG TCK clock pulse at power-on\nIO14 (TMS): pull-up causes JTAG to reset state if accidental TCK pulse\nIO15 (TDO): pull up for debug output, down for fast/quiet boot (internal pull-up)\nIO12 (TDI):  pull up for 1.8V flash, down for 3.3V flash (internal pull-down)
 Connection ~ 2950 7300
 $Comp
@@
 F 2 "stdpads:R_0805" H 2350 6500 50  0001 C CNN
 F 3 "~" H 2350 6500 50  0001 C CNN
-F 4 "C31850" H 2350 6500 50  0001 C CNN "LCSC Part"
+F 4 "C17414" H 2350 6500 50  0001 C CNN "LCSC Part"
 	1    2350 6500
 	1    0    0    -1
@@
 F 2 "stdpads:R_0805" H 2350 7200 50  0001 C CNN
 F 3 "~" H 2350 7200 50  0001 C CNN
-F 4 "C21190" H 2350 7200 50  0001 C CNN "LCSC Part"
+F 4 "C17513" H 2350 7200 50  0001 C CNN "LCSC Part"
 	1    2350 7200
 	1    0    0    -1
@@
 F 2 "stdpads:R_0805" H 2050 7200 50  0001 C CNN
 F 3 "~" H 2050 7200 50  0001 C CNN
-F 4 "C31850" H 2050 7200 50  0001 C CNN "LCSC Part"
+F 4 "C17414" H 2050 7200 50  0001 C CNN "LCSC Part"
 	1    2050 7200
 	1    0    0    -1
@@
 F 2 "stdpads:R_0805" H 2050 6500 50  0001 C CNN
 F 3 "~" H 2050 6500 50  0001 C CNN
-F 4 "C31850" H 2050 6500 50  0001 C CNN "LCSC Part"
+F 4 "C17414" H 2050 6500 50  0001 C CNN "LCSC Part"
 	1    2050 6500
 	1    0    0    -1
@@
 F 2 "stdpads:R_0805" H 4250 1450 50  0001 C CNN
 F 3 "~" H 4250 1450 50  0001 C CNN
+F 4 "C17414" H 4250 1450 50  0001 C CNN "LCSC Part"
 	1    4250 1450
 	-1   0    0    -1
@@
 F 2 "stdpads:C_0805" H 4250 1650 50  0001 C CNN
 F 3 "~" H 4250 1650 50  0001 C CNN
+F 4 "C28233" H 4250 1650 50  0001 C CNN "LCSC Part"
 	1    4250 1650
 	-1   0    0    -1
@@
 F 2 "stdpads:R_0805" H 1250 2750 50  0001 C CNN
 F 3 "~" H 1250 2750 50  0001 C CNN
-F 4 "C25190" H 1250 2750 50  0001 C CNN "LCSC Part"
+F 4 "C17408" H 1250 2750 50  0001 C CNN "LCSC Part"
 	1    1250 2750
 	0    -1   -1   0
@@
 N~CS~
 Text Notes 4400 2650 2    50   ~ 0
-internal weak pulldown on IO12
+internal pulldown on IO12
 Text Notes 4400 2550 2    50   ~ 0
-internal weak pullup on IO14
+internal pullup on IO14, toggles at boot
 Text Notes 4400 2850 2    50   ~ 0
-internal weak pulldown on IO13
+internal pulldown on IO13
 Wire Wire Line
 	4650 2750 4650 2950
@@
 F 2 "stdpads:R_0805" H 3500 1950 50  0001 C CNN
 F 3 "~" H 3500 1950 50  0001 C CNN
-F 4 "C25190" H 3500 1950 50  0001 C CNN "LCSC Part"
+F 4 "C17513" H 3500 1950 50  0001 C CNN "LCSC Part"
 	1    3500 1950
 	0    -1   1    0
@@
 F 2 "stdpads:R_0805" H 3200 2050 50  0001 C CNN
 F 3 "~" H 3200 2050 50  0001 C CNN
-F 4 "C21190" H 3200 2050 50  0001 C CNN "LCSC Part"
+F 4 "C17513" H 3200 2050 50  0001 C CNN "LCSC Part"
 	1    3200 2050
 	1    0    0    -1
@@
 F 2 "stdpads:C_0805" H 7200 4650 50  0001 C CNN
 F 3 "~" H 7200 4650 50  0001 C CNN
+F 4 "C15850" H 7200 4650 50  0001 C CNN "LCSC Part"
 	1    7200 4650
 	-1   0    0    -1
@@
 F 2 "stdpads:C_0805" H 7600 4650 50  0001 C CNN
 F 3 "~" H 7600 4650 50  0001 C CNN
+F 4 "C15850" H 7600 4650 50  0001 C CNN "LCSC Part"
 	1    7600 4650
 	-1   0    0    -1
@@
 F 2 "stdpads:C_0805" H 8000 4650 50  0001 C CNN
 F 3 "~" H 8000 4650 50  0001 C CNN
+F 4 "C15850" H 8000 4650 50  0001 C CNN "LCSC Part"
 	1    8000 4650
 	-1   0    0    -1
@@
 	6550 2650 6850 2650
 Text Notes 6900 2550 0    50   ~ 0
-internal weak pulldown on IO4
+internal pulldown on IO4
 Text Notes 6900 2650 0    50   ~ 0
-internal weak pullup on IO0
+internal pullup on IO0, toggles at boot
 Text Notes 6900 2750 0    50   ~ 0
-internal weak pulldown on IO2
+internal pulldown on IO2
 Text Notes 6900 2850 0    50   ~ 0
-internal weak pullup on IO15
+internal pullup on IO15, toggles at boot
 Text Notes 6900 2300 0    50   ~ 0
-internal weak pullup on IO5
+internal pullup on IO5, toggles at boot
 NoConn ~ 4750 1950
-$Comp
-L Device:R_Small R22
-U 1 1 6869399E
-P 4850 5500
-F 0 "R22" V 4700 5500 50  0000 C CNN
-F 1 "1k" V 4800 5500 50  0000 C BNN
-F 2 "stdpads:R_0805" H 4850 5500 50  0001 C CNN
-F 3 "~" H 4850 5500 50  0001 C CNN
-F 4 "C25190" H 4850 5500 50  0001 C CNN "LCSC Part"
-	1    4850 5500
-	0    1    1    0
-$EndComp
 Wire Wire Line
 	2200 5100 2600 5100
@@
 F 2 "stdpads:R_0805" H 6950 1850 50  0001 C CNN
 F 3 "~" H 6950 1850 50  0001 C CNN
-F 4 "C25190" H 6950 1850 50  0001 C CNN "LCSC Part"
+F 4 "C17561" H 6950 1850 50  0001 C CNN "LCSC Part"
 	1    6950 1850
 	0    -1   1    0
@@
 F 2 "stdpads:R_0805" H 6950 1550 50  0001 C CNN
 F 3 "~" H 6950 1550 50  0001 C CNN
-F 4 "C25190" H 6950 1550 50  0001 C CNN "LCSC Part"
+F 4 "C17561" H 6950 1550 50  0001 C CNN "LCSC Part"
 	1    6950 1550
 	0    -1   1    0
@@
 F 2 "stdpads:R_0805" H 6950 2150 50  0001 C CNN
 F 3 "~" H 6950 2150 50  0001 C CNN
-F 4 "C25190" H 6950 2150 50  0001 C CNN "LCSC Part"
+F 4 "C17561" H 6950 2150 50  0001 C CNN "LCSC Part"
 	1    6950 2150
 	0    -1   1    0
@@
 F 2 "stdpads:C_0805" H 8400 4650 50  0001 C CNN
 F 3 "~" H 8400 4650 50  0001 C CNN
+F 4 "C15850" H 8400 4650 50  0001 C CNN "LCSC Part"
 	1    8400 4650
 	-1   0    0    -1
@@
 	8400 4750 8000 4750
 Connection ~ 8400 4750
+$Comp
+L Device:R_Small R36
+U 1 1 626EB58A
+P 9450 4150
+AR Path="/64084316/626EB58A" Ref="R36"  Part="1"
+AR Path="/61C6168C/626EB58A" Ref="R?"  Part="1"
+F 0 "R36" H 9509 4196 50  0000 L CNN
+F 1 "10k" H 9509 4105 50  0000 L CNN
+F 2 "stdpads:R_0805" H 9450 4150 50  0001 C CNN
+F 3 "~" H 9450 4150 50  0001 C CNN
+F 4 "C17414" H 9450 4150 50  0001 C CNN "LCSC Part"
+	1    9450 4150
+	-1   0    0    -1
+$EndComp
+$Comp
+L power:+3V3 #PWR?
+U 1 1 626EB590
+P 9450 3550
+AR Path="/626EB590" Ref="#PWR?"  Part="1"
+AR Path="/61C6168C/626EB590" Ref="#PWR?"  Part="1"
+AR Path="/64084316/626EB590" Ref="#PWR0235"  Part="1"
+F 0 "#PWR0235" H 9450 3400 50  0001 C CNN
+F 1 "+3V3" H 9450 3700 50  0000 C CNN
+F 2 "" H 9450 3550 50  0001 C CNN
+F 3 "" H 9450 3550 50  0001 C CNN
+	1    9450 3550
+	1    0    0    -1
+$EndComp
+Wire Wire Line
+	9150 3850 9550 3850
+Text HLabel 9550 3750 2    50   Output ~ 0
+N~CS~
+$Comp
+L Device:R_Small R35
+U 1 1 626EDF1A
+P 9450 3650
+AR Path="/64084316/626EDF1A" Ref="R35"  Part="1"
+AR Path="/61C6168C/626EDF1A" Ref="R?"  Part="1"
+F 0 "R35" H 9509 3696 50  0000 L CNN
+F 1 "10k" H 9509 3605 50  0000 L CNN
+F 2 "stdpads:R_0805" H 9450 3650 50  0001 C CNN
+F 3 "~" H 9450 3650 50  0001 C CNN
+F 4 "C17414" H 9450 3650 50  0001 C CNN "LCSC Part"
+	1    9450 3650
+	-1   0    0    -1
+$EndComp
+Wire Wire Line
+	9550 3750 9450 3750
+Text HLabel 9550 3850 2    50   Input ~ 0
+WRCLK
+Text HLabel 9550 3950 2    50   Output ~ 0
+RDCLK
+Wire Wire Line
+	9450 4050 9450 3950
+Wire Wire Line
+	9450 3950 9550 3950
+$Comp
+L power:GND #PWR0236
+U 1 1 6271322C
+P 9450 4250
+F 0 "#PWR0236" H 9450 4000 50  0001 C CNN
+F 1 "GND" H 9450 4100 50  0000 C CNN
+F 2 "" H 9450 4250 50  0001 C CNN
+F 3 "" H 9450 4250 50  0001 C CNN
+	1    9450 4250
+	1    0    0    -1
+$EndComp
+$Comp
+L Device:R_Small R34
+U 1 1 6272457D
+P 9150 3650
+AR Path="/64084316/6272457D" Ref="R34"  Part="1"
+AR Path="/61C6168C/6272457D" Ref="R?"  Part="1"
+F 0 "R34" H 9209 3696 50  0000 L CNN
+F 1 "10k" H 9209 3605 50  0000 L CNN
+F 2 "stdpads:R_0805" H 9150 3650 50  0001 C CNN
+F 3 "~" H 9150 3650 50  0001 C CNN
+F 4 "C17414" H 9150 3650 50  0001 C CNN "LCSC Part"
+	1    9150 3650
+	-1   0    0    -1
+$EndComp
+Wire Wire Line
+	9150 3750 9150 3850
+Wire Wire Line
+	9150 3550 9450 3550
+Connection ~ 9450 3550
+$Comp
+L Device:R_Small R22
+U 1 1 62C2CF67
+P 4850 5500
+F 0 "R22" V 4700 5500 50  0000 C CNN
+F 1 "10k" V 4800 5500 50  0000 C BNN
+F 2 "stdpads:R_0805" H 4850 5500 50  0001 C CNN
+F 3 "~" H 4850 5500 50  0001 C CNN
+F 4 "C17414" H 4850 5500 50  0001 C CNN "LCSC Part"
+	1    4850 5500
+	0    -1   1    0
+$EndComp
 $EndSCHEMATC
