File: NuBus-ESP32.sch (KiCad schematic (older format))
At the start: 21 parts, among them J2 Xunpu TF-115, J3 microUSB-B, U27 AZ1117EH-3.3TRG1

Commit message: Export gerbers just to test
Parts:
- C4, C5: LCSC Part (none) -> C15850
- J3: LCSC Part (none) -> C404969
- R1, R2, R4, R5: LCSC Part C25190 -> C17408
- R3: value 100 -> 22; LCSC Part C25190 -> C17561
- R6, R7: LCSC Part C25819 -> C17713
- U27: LCSC Part (none) -> C108494
Changed lines of the file:
@@
 F 2 "stdpads:R_0805" H 5750 3350 50  0001 C CNN
 F 3 "~" H 5750 3350 50  0001 C CNN
-F 4 "C25190" H 5750 3350 50  0001 C CNN "LCSC Part"
+F 4 "C17408" H 5750 3350 50  0001 C CNN "LCSC Part"
 	1    5750 3350
 	0    -1   1    0
@@
 F 2 "stdpads:R_0805" H 5750 3550 50  0001 C CNN
 F 3 "~" H 5750 3550 50  0001 C CNN
-F 4 "C25190" H 5750 3550 50  0001 C CNN "LCSC Part"
+F 4 "C17408" H 5750 3550 50  0001 C CNN "LCSC Part"
 	1    5750 3550
 	0    -1   -1   0
@@
 F 2 "stdpads:R_0805" H 6350 3400 50  0001 C CNN
 F 3 "~" H 6350 3400 50  0001 C CNN
-F 4 "C25819" H 6350 3400 50  0001 C CNN "LCSC Part"
+F 4 "C17713" H 6350 3400 50  0001 C CNN "LCSC Part"
 	1    6350 3400
 	1    0    0    -1
@@
 F 2 "stdpads:R_0805" H 6650 3400 50  0001 C CNN
 F 3 "~" H 6650 3400 50  0001 C CNN
-F 4 "C25819" H 6650 3400 50  0001 C CNN "LCSC Part"
+F 4 "C17713" H 6650 3400 50  0001 C CNN "LCSC Part"
 	1    6650 3400
 	1    0    0    -1
@@
 F 2 "stdpads:R_0805" H 5750 4250 50  0001 C CNN
 F 3 "~" H 5750 4250 50  0001 C CNN
-F 4 "C25190" H 5750 4250 50  0001 C CNN "LCSC Part"
+F 4 "C17408" H 5750 4250 50  0001 C CNN "LCSC Part"
 	1    5750 4250
 	0    -1   -1   0
@@
 F 2 "stdpads:R_0805" H 5750 4050 50  0001 C CNN
 F 3 "~" H 5750 4050 50  0001 C CNN
-F 4 "C25190" H 5750 4050 50  0001 C CNN "LCSC Part"
+F 4 "C17408" H 5750 4050 50  0001 C CNN "LCSC Part"
 	1    5750 4050
 	0    -1   -1   0
@@
 AR Path="/619A511F" Ref="R3"  Part="1"
 F 0 "R3" V 5600 3850 50  0000 C CNN
-F 1 "100" V 5700 3850 50  0000 C BNN
+F 1 "22" V 5700 3850 50  0000 C BNN
 F 2 "stdpads:R_0805" H 5750 3850 50  0001 C CNN
 F 3 "~" H 5750 3850 50  0001 C CNN
-F 4 "C25190" H 5750 3850 50  0001 C CNN "LCSC Part"
+F 4 "C17561" H 5750 3850 50  0001 C CNN "LCSC Part"
 	1    5750 3850
 	0    -1   1    0
@@
 F 2 "stdpads:USB_Micro-B_ShouHan_MicroXNJ" H 7250 4900 50  0001 C CNN
 F 3 "~" H 7250 4900 50  0001 C CNN
+F 4 "C404969" H 7100 4950 50  0001 C CNN "LCSC Part"
 	1    7100 4950
 	-1   0    0    -1
@@
 F 2 "stdpads:SOT-223" H 7400 2300 50  0001 C CNN
 F 3 "http://www.diodes.com/datasheets/AP1117.pdf" H 7500 1850 50  0001 C CNN
+F 4 "C108494" H 7400 2100 50  0001 C CNN "LCSC Part"
 	1    7400 2100
 	1    0    0    -1
@@
 F 2 "stdpads:C_0805" H 6900 2250 50  0001 C CNN
 F 3 "~" H 6900 2250 50  0001 C CNN
+F 4 "C15850" H 6900 2250 50  0001 C CNN "LCSC Part"
 	1    6900 2250
 	1    0    0    -1
@@
 F 2 "stdpads:C_0805" H 7900 2250 50  0001 C CNN
 F 3 "~" H 7900 2250 50  0001 C CNN
+F 4 "C15850" H 7900 2250 50  0001 C CNN "LCSC Part"
 	1    7900 2250
 	-1   0    0    -1
