File: NuBus.sch (KiCad schematic (older format))
At the start: 3 parts, among them J1 MacNuBus

Commit message: Export gerbers just to test
Parts:
- C34, C35: LCSC Part (none) -> C15850
Changed lines of the file:
@@
 F 2 "stdpads:C_0805" H 6450 4050 50  0001 C CNN
 F 3 "~" H 6450 4050 50  0001 C CNN
+F 4 "C15850" H 6450 4050 50  0001 C CNN "LCSC Part"
 	1    6450 4050
 	-1   0    0    -1
@@
 F 2 "stdpads:C_0805" H 6050 4050 50  0001 C CNN
 F 3 "~" H 6050 4050 50  0001 C CNN
+F 4 "C15850" H 6050 4050 50  0001 C CNN "LCSC Part"
 	1    6050 4050
 	-1   0    0    -1
