File: ROM.sch (KiCad schematic (older format))
At the start: 6 parts, among them U2 SST39SF040, U28 SST39SF040, U4 74LVC245AD

Commit message: Export gerbers just to test
Parts:
- C16, C17, C18: LCSC Part (none) -> C15850
- U2: LCSC Part (none) -> C72257
- U28: LCSC Part (none) -> C72128
- U4: LCSC Part (none) -> C6080
Changed lines of the file:
@@
 F 2 "stdpads:PLCC-32_SMDSocket" H 5050 2600 50  0001 C CNN
 F 3 "http://ww1.microchip.com/downloads/en/DeviceDoc/20005022C.pdf" H 5050 3650 50  0001 C CNN
+F 4 "C72257" H 5050 3650 50  0001 C CNN "LCSC Part"
 	1    5050 3650
 	1    0    0    -1
@@
 F 2 "Package_DIP:DIP-32_W15.24mm_Socket_LongPads" H 5050 4800 50  0001 C CNN
 F 3 "http://ww1.microchip.com/downloads/en/DeviceDoc/20005022C.pdf" H 5050 5850 50  0001 C CNN
+F 4 "C72128" H 5050 5850 50  0001 C CNN "LCSC Part"
 	1    5050 5850
 	1    0    0    -1
@@
 F 2 "stdpads:SOIC-20W_7.5mm" H 6550 2550 50  0001 C TNN
 F 3 "" H 6550 3300 60  0001 C CNN
+F 4 "C6080" H 6550 3200 50  0001 C CNN "LCSC Part"
 	1    6550 3200
 	-1   0    0    -1
@@
 F 2 "stdpads:C_0805" H 7150 5000 50  0001 C CNN
 F 3 "~" H 7150 5000 50  0001 C CNN
+F 4 "C15850" H 7150 5000 50  0001 C CNN "LCSC Part"
 	1    7150 5000
 	-1   0    0    -1
@@
 F 2 "stdpads:C_0805" H 6750 5000 50  0001 C CNN
 F 3 "~" H 6750 5000 50  0001 C CNN
+F 4 "C15850" H 6750 5000 50  0001 C CNN "LCSC Part"
 	1    6750 5000
 	-1   0    0    -1
@@
 F 2 "stdpads:C_0805" H 7550 5000 50  0001 C CNN
 F 3 "~" H 7550 5000 50  0001 C CNN
+F 4 "C15850" H 7550 5000 50  0001 C CNN "LCSC Part"
 	1    7550 5000
 	-1   0    0    -1
