File: DataReg.kicad_sch (KiCad schematic)
At the start: 39 parts, among them U10 74LVC574AD, U11 74LVC574AD, U12 74LVC574AD, U13 74LVC574AD, U29 74LVC574AD, U30 74LVC574AD, U31 74LVC574AD, U32 74LVC574AD, U33 74LVC574AD, U35 74LVC74AD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

Commit message: Prototype with 74xx
Parts:
- added R37: 1k, stdpads:R_0805, symbol Device:R_Small
Connections:
- net +3V3: now also U35.10 (~{S}), U35.13 (~{R}), R37.1; no longer U35.1 (~{R}), U35.4 (~{S})
- net MISO: now also U35.8 (~{Q}); no longer U35.6 (~{Q})
- net SCK: now also U35.11 (C); no longer U35.3 (C)
- net WRCLK: no longer U5.1 (~{OE}), U6.1 (~{OE}), U7.1 (~{OE}), U8.1 (~{OE}), U9.1 (~{OE})
- net at U29.2 (D0), U5.19 (Q0): now also R37.2
- net at U33.12 (Q7): now also U35.12 (D); no longer U35.2 (D)
- new net P~{OE}: U5.1 (~{OE}), U6.1 (~{OE}), U7.1 (~{OE}), U8.1 (~{OE}), U9.1 (~{OE})
