File: NuBus-ESP32.kicad_pcb (KiCad board)
At the start: 4 copper layers, 193.7 x 101.6 mm, 151 parts, among them J1 MacNuBus, J2 Xunpu TF-115, J3 microUSB-B, J4 JTAG, Q1 MMBT3904, Q2 MMBT3904, Q3 MMBT3904, Q4 MMBT3904, Q5 MMBT3904, U1 ESP-WROVER-32, U10 74LVC574AD, U11 74LVC574AD, U12 74LVC574AD, U13 74LVC574AD, U14 74LVC574AD, U15 74LVC574AD, U16 74LVC574AD, U17 74LVC74AD, U18 74LVC74AD, U19 74LVC74AD, U2 SST39SF040, U20 74LVC86AD, U21 74LVC32AD, U22 74LVC02AD, U23 74LVC00AD, U24 74LVC125AD, U25 74LVC32AD, U26 74LVC125AD, U27 AZ1117EH-3.3TRG1, U28 SST39SF040, U29 74LVC574AD, U3 CH340G, U30 74LVC574AD, U31 74LVC574AD, U32 74LVC574AD, U33 74LVC574AD, U34 74LVC32AD, U35 74LVC74AD, U36 74LVC74AD, U37 74LVC74AD, U38 74LVC574AD, U39 74LVC574AD, U4 74LVC245AD, U40 74LVC574AD, U41 74LVC574AD, U42 74LVC32AD, U5 74LVC574AD, U6 74LVC574AD, U7 74LVC574AD, U8 74LVC574AD, U9 74LVC574AD, Y1 12M

Commit message: idk
Parts:
- removed C13, C14, C18, C19, C20, C21, C22, C23, C24, C25, C26, C27, C28, C29, C30, C31, C32, C33, C36, C37, C38, C39, C4, C40, C41, C42, C43, C44, C45, C46, C47, C48, C49, C50, C6: 10u, stdpads:C_0805
- removed C2: 22p, stdpads:C_0805
- removed C3: 100n, stdpads:C_0805
- removed FID5: Fiducial, stdpads:Fiducial
- removed Q1, Q2, Q3, Q4, Q5: MMBT3904, stdpads:SOT-23
- removed R15: 100, stdpads:R_0805
- removed R16, R22, R28, R29, R30, R34, R35, R36, R38: 10k, stdpads:R_0805
- removed R21, R23, R24: DNP, stdpads:R_0805
- removed R25, R26, R33: 22, stdpads:R_0805
- removed R27, R31, R32, R37: 1k, stdpads:R_0805
- removed the U10 at (108.6, 67.3)
- removed U19, U35, U36, U37: 74LVC74AD, stdpads:SOIC-14_3.9mm
- removed U20: 74LVC86AD, stdpads:SOIC-14_3.9mm
- removed U21, U25, U34, U42: 74LVC32AD, stdpads:SOIC-14_3.9mm
- removed U22: 74LVC02AD, stdpads:SOIC-14_3.9mm
- removed U23: 74LVC00AD, stdpads:SOIC-14_3.9mm
- removed U24, U26: 74LVC125AD, stdpads:SOIC-14_3.9mm
- removed U27: AZ1117EH-3.3TRG1, stdpads:SOT-223
- removed U28: SST39SF040, Package_DIP:DIP-32_W15.24mm_Socket_LongPads
- removed U29, U30, U31, U32, U33, U38, U39, U40, U41: 74LVC574AD, stdpads:SOIC-20W_7.5mm
- removed the U7 at (139.1, 97.8)
- removed the U8 at (154.3, 97.8)
- removed the U9 at (169.5, 97.8)
- removed Y1: 12M, stdpads:Crystal_HC49-SMD
- added D1: Schottky, stdpads:D_SOD-323, F.Cu at (8.14, 24.1)
- added J2: UART, stdpads:Tag-Connect_TC2030-IDC-NL_2x03_P1.27mm_Vertical_with_bottom_clip, F.Cu at (17.9, 12.6)
- added J6: FJTAG, stdpads:Tag-Connect_TC2050-IDC-NL_2x05_P1.27mm_Vertical_with_bottom_clip, F.Cu at (8.12, 5.96)
- added REF**: R_0603, stdpads:R_0603, F.Cu at (220.5, 79.6)
- added REF**: R_0603, stdpads:R_0603, F.Cu at (220.5, 90.9)
- added REF**: R_0603, stdpads:R_0603, F.Cu at (222.6, 84.5)
- added REF**: R_0603, stdpads:R_0603, F.Cu at (220.5, 81.0)
- added REF**: DSUB-15-HD_Female_Horizontal_P2.29x1.98mm_EdgePinOffset3.03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, Connector_Dsub:DSUB-15-HD_Female_Horizontal_P2.29x1.98mm_EdgePinOffset3.03mm_Housed_MountingHolesOffset4.94mm, F.Cu at (229.3, 87.8)
- added REF**: R_0603, stdpads:R_0603, F.Cu at (222.6, 109.9)
- added REF**: R_0603, stdpads:R_0603, F.Cu at (220.5, 103.6)
- added REF**: R_0603, stdpads:R_0603, F.Cu at (222.6, 107.1)
- added REF**: R_0603, stdpads:R_0603, F.Cu at (220.5, 102.2)
- added REF**: R_0603, stdpads:R_0603, F.Cu at (220.5, 93.7)
- added REF**: R_0603, stdpads:R_0603, F.Cu at (222.6, 87.3)
- added REF**: R_0603, stdpads:R_0603, F.Cu at (220.5, 86.6)
- added REF**: R_0603, stdpads:R_0603, F.Cu at (224.0, 97.2)
- added REF**: R_0603, stdpads:R_0603, F.Cu at (208.4, 69.8)
- added REF**: R_0603, stdpads:R_0603, F.Cu at (220.5, 110.6)
- added REF**: R_0603, stdpads:R_0603, F.Cu at (224.0, 102.9)
- added REF**: R_0603, stdpads:R_0603, F.Cu at (220.5, 107.8)
- added REF**: R_0603, stdpads:R_0603, F.Cu at (224.0, 85.9)
- added REF**: R_0603, stdpads:R_0603, F.Cu at (220.5, 95.1)
- added REF**: R_0603, stdpads:R_0603, F.Cu at (220.5, 106.4)
- added REF**: R_0603, stdpads:R_0603, F.Cu at (201.5, 54.7)
- added REF**: R_0603, stdpads:R_0603, F.Cu at (220.5, 97.9)
- added REF**: R_0603, stdpads:R_0603, F.Cu at (220.5, 82.4)
- added REF**: R_0603, stdpads:R_0603, F.Cu at (224.0, 83.1)
- added REF**: R_0603, stdpads:R_0603, F.Cu at (222.6, 90.2)
- added REF**: R_0603, stdpads:R_0603, F.Cu at (224.0, 100.0)
- added REF**: R_0603, stdpads:R_0603, F.Cu at (222.6, 101.5)
- added REF**: R_0603, stdpads:R_0603, F.Cu at (200.8, 57.9)
- added REF**: L_Changjiang_FNR4015S, Inductor_SMD:L_Changjiang_FNR4015S, F.Cu at (181.9, 129.4)
- added REF**: R_0603, stdpads:R_0603, F.Cu at (220.5, 96.5)
- added REF**: R_0603, stdpads:R_0603, F.Cu at (224.0, 105.7)
- added REF**: R_0603, stdpads:R_0603, F.Cu at (224.0, 88.7)
- added REF**: R_0603, stdpads:R_0603, F.Cu at (224.0, 80.3)
- added REF**: R_0603, stdpads:R_0603, F.Cu at (181.2, 126.2)
- added REF**: R_0603, stdpads:R_0603, F.Cu at (220.5, 88.0)
- added REF**: R_0603, stdpads:R_0603, F.Cu at (220.5, 89.5)
- added REF**: R_0603, stdpads:R_0603, F.Cu at (222.6, 81.7)
- added REF**: L_Changjiang_FNR4015S, Inductor_SMD:L_Changjiang_FNR4015S, F.Cu at (194.4, 129.4)
- added REF**: R_0603, stdpads:R_0603, F.Cu at (220.5, 92.3)
- added REF**: R_0603, stdpads:R_0603, F.Cu at (220.5, 100.8)
- added REF**: R_0603, stdpads:R_0603, F.Cu at (220.5, 109.2)
- added REF**: R_0603, stdpads:R_0603, F.Cu at (222.6, 104.3)
- added REF**: R_0603, stdpads:R_0603, F.Cu at (220.5, 78.2)
- added REF**: R_0603, stdpads:R_0603, F.Cu at (220.5, 105.0)
- added REF**: R_0603, stdpads:R_0603, F.Cu at (220.5, 83.8)
- added REF**: R_0603, stdpads:R_0603, F.Cu at (222.6, 78.9)
- added REF**: R_0603, stdpads:R_0603, F.Cu at (224.0, 91.6)
- added REF**: R_0603, stdpads:R_0603, F.Cu at (200.8, 59.3)
- added REF**: R_0603, stdpads:R_0603, F.Cu at (222.6, 93.0)
- added REF**: R_0603, stdpads:R_0603, F.Cu at (222.6, 98.6)
- added REF**: SOT-223, stdpads:SOT-223, F.Cu at (83.8, 97.8)
- added REF**: C_0402, stdpads:C_0402, B.Cu at (132.8, 116.0)
- added REF**: C_0402, stdpads:C_0402, B.Cu at (143.0, 116.0)
- added REF**: R_0603, stdpads:R_0603, F.Cu at (220.5, 99.3)
- added REF**: C_0402, stdpads:C_0402, B.Cu at (158.0, 136.2)
- added REF**: C_0402, stdpads:C_0402, B.Cu at (113.7, 92.0)
- added REF**: C_0402, stdpads:C_0402, B.Cu at (154.4, 136.2)
- added REF**: C_0402, stdpads:C_0402, B.Cu at (131.1, 99.3)
- added REF**: C_0402, stdpads:C_0402, B.Cu at (112.5, 116.0)
- added REF**: C_0402, stdpads:C_0402, B.Cu at (110.0, 92.0)
- added REF**: C_0402, stdpads:C_0402, B.Cu at (127.8, 95.4)
- added REF**: C_0402, stdpads:C_0402, B.Cu at (153.2, 116.0)
- added REF**: C_0402, stdpads:C_0402, B.Cu at (146.8, 136.2)
- added REF**: C_0402, stdpads:C_0402, B.Cu at (134.2, 99.2)
- added REF**: R_0603, stdpads:R_0603, F.Cu at (224.0, 94.4)
- added REF**: C_0402, stdpads:C_0402, B.Cu at (132.3, 94.1)
- added REF**: C_0402, stdpads:C_0402, B.Cu at (131.9, 97.3)
- added REF**: C_0402, stdpads:C_0402, B.Cu at (99.3, 92.0)
- added REF**: C_0402, stdpads:C_0402, B.Cu at (150.4, 136.2)
- added REF**: C_0402, stdpads:C_0402, B.Cu at (122.7, 116.0)
- added REF**: C_0402, stdpads:C_0402, B.Cu at (106.9, 116.0)
- added REF**: C_0402, stdpads:C_0402, B.Cu at (129.8, 94.1)
- added REF**: C_0402, stdpads:C_0402, B.Cu at (89.6, 116.0)
- added REF**: C_0402, stdpads:C_0402, B.Cu at (117.5, 92.0)
- added REF**: C_0402, stdpads:C_0402, B.Cu at (133.9, 97.3)
- added REF**: R_0603, stdpads:R_0603, F.Cu at (220.5, 85.2)
- added REF**: C_0402, stdpads:C_0402, B.Cu at (122.8, 83.9)
- added REF**: C_0402, stdpads:C_0402, B.Cu at (94.5, 136.2)
- added REF**: C_0402, stdpads:C_0402, B.Cu at (90.9, 136.2)
- added REF**: C_0402, stdpads:C_0402, B.Cu at (110.0, 102.7)
- added REF**: C_0402, stdpads:C_0402, B.Cu at (120.0, 92.0)
- added REF**: C_0402, stdpads:C_0402, B.Cu at (83.8, 116.0)
- added REF**: C_0402, stdpads:C_0402, B.Cu at (129.1, 100.5)
- added REF**: C_0402, stdpads:C_0402, B.Cu at (105.6, 102.7)
- added REF**: C_0402, stdpads:C_0402, B.Cu at (133.1, 100.5)
- added REF**: C_0402, stdpads:C_0402, B.Cu at (129.2, 97.3)
- added REF**: R_0603, stdpads:R_0603, F.Cu at (222.6, 95.8)
- added REF**: C_0402, stdpads:C_0402, B.Cu at (115.1, 102.7)
- added REF**: C_0402, stdpads:C_0402, B.Cu at (119.2, 83.2)
- added REF**: C_0402, stdpads:C_0402, B.Cu at (131.1, 95.4)
- added REF**: C_0402, stdpads:C_0402, B.Cu at (127.8, 98.6)
- added REF**: C_0402, stdpads:C_0402, B.Cu at (215.6, 52.8)
- added REF**: C_0402, stdpads:C_0402, B.Cu at (134.2, 95.4)
- added REF**: C_0402, stdpads:C_0402, B.Cu at (95.4, 116.0)
- added REF**: C_0402, stdpads:C_0402, B.Cu at (88.4, 136.2)
- added REF**: C_0402, stdpads:C_0402, B.Cu at (101.1, 116.0)
- added REF**: C_0402, stdpads:C_0402, B.Cu at (161.8, 116.0)
- added U10: 74LVC245APW, stdpads:TSSOP-20_4.4x6.5mm_P0.65mm, F.Cu at (114.9, 118.5)
- added U10: 74LVC245APW, stdpads:TSSOP-20_4.4x6.5mm_P0.65mm, F.Cu at (215.0, 110.8)
- added U59: TPS62A01, stdpads:SOT-563, F.Cu at (178.0, 128.6)
- added U59: TPS62A01, stdpads:SOT-563, F.Cu at (190.5, 128.7)
- added U7: 74LVC245APW, stdpads:TSSOP-20_4.4x6.5mm_P0.65mm, F.Cu at (215.0, 81.0)
- added U7: 74LVC245APW, stdpads:TSSOP-20_4.4x6.5mm_P0.65mm, F.Cu at (145.4, 118.5)
- added U8: 74LVC245APW, stdpads:TSSOP-20_4.4x6.5mm_P0.65mm, F.Cu at (215.0, 92.3)
- added U8: 74LVC245APW, stdpads:TSSOP-20_4.4x6.5mm_P0.65mm, F.Cu at (135.3, 118.5)
- added U9: 74LVC245APW, stdpads:TSSOP-20_4.4x6.5mm_P0.65mm, F.Cu at (125.1, 118.5)
- added U9: 74LVC245APW, stdpads:TSSOP-20_4.4x6.5mm_P0.65mm, F.Cu at (215.0, 103.7)
- added Y2: 25M, stdpads:Crystal_SMD_3225-4Pin_3.2x2.5mm, F.Cu at (115.1, 83.7)
- C1: value 22p -> 100n; footprint stdpads:C_0805 -> stdpads:C_0402
- C10, C15, C5, C8: value 10u -> 100n; footprint stdpads:C_0805 -> stdpads:C_0402; moved to B.Cu
- C11, C12: value 10u -> 4u7
- C16, C17: value 10u -> 120p; footprint stdpads:C_0805 -> stdpads:C_0402
- C7, C9: value 10u -> 22u
- H1, H2, H3, H4: value (none) -> ~
- J3: value microUSB-B -> microUSB; footprint stdpads:USB_Micro-B_ShouHan_MicroXNJ -> stdpads:USB_Micro-B_Amphenol_10118192-0001
- J4: value JTAG -> EJTAG; footprint Connector_IDC:IDC-Header_2x05_P2.54mm_Vertical -> stdpads:Tag-Connect_TC2050-IDC-NL_2x05_P1.27mm_Vertical_with_bottom_clip
- J5: renamed from J2; value Xunpu TF-115 -> microSD
- R1, R12, R2, R5, R8: value 100 -> 33; footprint stdpads:R_0805 -> stdpads:R_0603
- R10: value 1k -> 3k3; footprint stdpads:R_0805 -> stdpads:R_0603
- R11, R4: value 100 -> 68; footprint stdpads:R_0805 -> stdpads:R_0603
- R13, R14: value 10k -> 68; footprint stdpads:R_0805 -> stdpads:R_0603
- R17: value 1k -> 15k; footprint stdpads:R_0805 -> stdpads:R_0603
- R18: value DNP -> 17k; footprint stdpads:R_0805 -> stdpads:R_0603
- R19: value 1k -> 56k; footprint stdpads:R_0805 -> stdpads:R_0603
- R20: value DNP -> 12k; footprint stdpads:R_0805 -> stdpads:R_0603
- R3: value 22 -> 33; footprint stdpads:R_0805 -> stdpads:R_0603
- R6, R7: value 47k -> 33; footprint stdpads:R_0805 -> stdpads:R_0603
- R9: value 22 -> 3k3; footprint stdpads:R_0805 -> stdpads:R_0603
- U1: value ESP-WROVER-32 -> LFE5U-12F-BG256; footprint stdpads:ESP32-WROVER_WROOM-32_WROVER -> stdpads:Lattice_CABGA-256_14x14mm
- U11, U12, U13, U5, U6: value 74LVC574AD -> 74LVC125APW; footprint stdpads:SOIC-20W_7.5mm -> stdpads:TSSOP-14_4.4x5mm_P0.65mm
- U14: value 74LVC574AD -> TPS22919; footprint stdpads:SOIC-20W_7.5mm -> stdpads:SOT-363
- U15: value 74LVC574AD -> TPD2EUSB30; footprint stdpads:SOIC-20W_7.5mm -> stdpads:TI_DRT-3
- U16: value 74LVC574AD -> Si5351A-B-GT; footprint stdpads:SOIC-20W_7.5mm -> stdpads:MSOP-10_3x3mm_P0.5mm
- U17, U18: value 74LVC74AD -> 74LVC125APW; footprint stdpads:SOIC-14_3.9mm -> stdpads:TSSOP-14_4.4x5mm_P0.65mm
- U2: value SST39SF040 -> ESP32-S2-MINI-2; footprint stdpads:PLCC-32_SMDSocket -> stdpads:ESP32-S2-MINI-1U
- U3: value CH340G -> W9825G6KH-6; footprint stdpads:SOIC-16_3.9mm -> stdpads:TSOP-II-54_22.2x10.16mm_P0.8mm
- U4: value 74LVC245AD -> W9825G6KH-6; footprint stdpads:SOIC-20W_7.5mm -> stdpads:TSOP-II-54_22.2x10.16mm_P0.8mm
- moved R1 247.7 mm to (16.3, -2.77)
- moved J3 246.1 mm to (7.34, 13.2)
- moved R10 236.7 mm to (3.74, 22.6)
- moved J4 228.1 mm to (8.12, -0.68)
- moved R13 221.2 mm to (26.9, 4.58)
- moved R14 216.4 mm to (16.3, 2.13), turned to 0 degrees
- moved C1 214.1 mm to (3.34, 24.9), turned to 0 degrees
- moved R7 200.6 mm to (26.9, -0.32), turned to 0 degrees
- moved R5 199.4 mm to (26.9, -2.77), turned to 0 degrees
- moved C34 178.9 mm to (24.2, 20.4)
- moved R9 176.8 mm to (3.74, 20.1), turned to 0 degrees
- moved U14 173.2 mm to (7.79, 20.8)
- moved U15 166.4 mm to (19.6, -2.77)
- moved R3 163.9 mm to (86.0, 113.8)
- moved R8 127.3 mm to (26.9, 2.13), turned to 0 degrees
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Connections:
- C1 pad 1: Net-(C1-Pad1) -> /IOP/Mac5Vsense
- C10 pad 1: +3V3 -> +5V
- C11 pad 1: +3V3 -> +5V
- C12 pad 1: +3V3 -> +5V
- C15 pad 1: +3V3 -> +5V
- C16 pad 1: +5V -> (no net)
- C16 pad 2: GND -> (no net)
- C17 pad 1: +5V -> +3V3
- C17 pad 2: GND -> (no net)
- C5 pad 1: +3V3 -> (no net)
- C7 pad 1: +3V3 -> (no net)
- J1 pad A10: /AddrLatch/~{AD}9 -> /NuBus/~{AD}9
- J1 pad A11: /AddrLatch/~{AD}11 -> /NuBus/~{AD}11
- J1 pad A12: /AddrLatch/~{AD}13 -> /NuBus/~{AD}13
- J1 pad A13: /AddrLatch/~{AD}15 -> /NuBus/~{AD}15
- J1 pad A14: /AddrLatch/~{AD}17 -> /NuBus/~{AD}17
- J1 pad A15: /AddrLatch/~{AD}19 -> /NuBus/~{AD}19
- J1 pad A16: /AddrLatch/~{AD}21 -> /NuBus/~{AD}21
- J1 pad A17: /AddrLatch/~{AD}23 -> /NuBus/~{AD}23
- J1 pad A18: /AddrLatch/~{AD}25 -> /NuBus/~{AD}25
- J1 pad A19: /AddrLatch/~{AD}27 -> /NuBus/~{AD}27
- J1 pad A20: /AddrLatch/~{AD}29 -> /NuBus/~{AD}29
- J1 pad A21: /AddrLatch/~{AD}31 -> /NuBus/~{AD}31
- J1 pad A24: unconnected-(J1-PadA24) -> /NuBus/~{ARB}1
- J1 pad A25: unconnected-(J1-PadA25) -> /NuBus/~{ARB}3
- J1 pad A26: /BusControl/~{ID}1 -> /NuBus/~{ID}1
- J1 pad A27: /BusControl/~{ID}3 -> /NuBus/~{ID}3
- J1 pad A28: /BusControl/~{ACK} -> /NuBus/~{ACK}
- J1 pad A30: unconnected-(J1-PadA30) -> /NuBus/~{RQST}
- J1 pad A31: /CtrlStatReg/~{NMRQ} -> /NuBus/~{NMRQ}
- J1 pad A5: /AddrLatch/~{TM}1 -> /NuBus/~{TM}1
- J1 pad A6: /AddrLatch/~{AD}1 -> /NuBus/~{AD}1
- J1 pad A7: /AddrLatch/~{AD}3 -> /NuBus/~{AD}3
- J1 pad A8: /AddrLatch/~{AD}5 -> /NuBus/~{AD}5
- J1 pad A9: /AddrLatch/~{AD}7 -> /NuBus/~{AD}7
- J1 pad C1: /CtrlStatReg/~{RES} -> /NuBus/~{RES}
- J1 pad C10: /AddrLatch/~{AD}8 -> /NuBus/~{AD}8
- J1 pad C11: /AddrLatch/~{AD}10 -> /NuBus/~{AD}10
- J1 pad C12: /AddrLatch/~{AD}12 -> /NuBus/~{AD}12
- J1 pad C13: /AddrLatch/~{AD}14 -> /NuBus/~{AD}14
- J1 pad C14: /AddrLatch/~{AD}16 -> /NuBus/~{AD}16
- J1 pad C15: /AddrLatch/~{AD}18 -> /NuBus/~{AD}18
- J1 pad C16: /AddrLatch/~{AD}20 -> /NuBus/~{AD}20
- J1 pad C17: /AddrLatch/~{AD}22 -> /NuBus/~{AD}22
- J1 pad C18: /AddrLatch/~{AD}24 -> /NuBus/~{AD}24
- J1 pad C19: /AddrLatch/~{AD}26 -> /NuBus/~{AD}26
- J1 pad C20: /AddrLatch/~{AD}28 -> /NuBus/~{AD}28
- J1 pad C21: /AddrLatch/~{AD}30 -> /NuBus/~{AD}30
- J1 pad C23: unconnected-(J1-PadC23) -> /NuBus/~{PFW}
- J1 pad C24: unconnected-(J1-PadC24) -> /NuBus/~{ARB}0
- J1 pad C25: unconnected-(J1-PadC25) -> /NuBus/~{ARB}2
- J1 pad C26: /BusControl/~{ID}0 -> /NuBus/~{ID}0
- J1 pad C27: /BusControl/~{ID}2 -> /NuBus/~{ID}2
- J1 pad C28: /BusControl/~{START} -> /NuBus/~{START}
- J1 pad C32: /AddrLatch/~{AD}[31..0] -> /NuBus/CLK
- J1 pad C5: /AddrLatch/~{TM}0 -> /NuBus/~{TM}0
- J1 pad C6: /AddrLatch/~{AD}0 -> /NuBus/~{AD}0
- J1 pad C7: /AddrLatch/~{AD}2 -> /NuBus/~{AD}2
- J1 pad C8: /AddrLatch/~{AD}4 -> /NuBus/~{AD}4
- J1 pad C9: /AddrLatch/~{AD}6 -> /NuBus/~{AD}6
- J3 pad 1: unconnected-(J3-Pad1) -> USB5V
- J3 pad 2: unconnected-(J3-Pad2) -> /D-
- J3 pad 3: unconnected-(J3-Pad3) -> /D+
- J4 pad 10: /ESP32/~{SRST} -> /E~{RES}
- J4 pad 2: /ESP32/TMS -> /ETMS
- J4 pad 4: Net-(J4-Pad4) -> /ETCK
- J4 pad 5: unconnected-(J4-Pad5) -> GND
- J4 pad 6: /ESP32/TDO -> /ETDO
- J4 pad 7: unconnected-(J4-Pad7) -> GND
- J4 pad 8: /ESP32/TDI -> /ETDI
- J4 pad 9: /ESP32/~{TRST} -> Net-(J4-Pin_9)
- J5 pad 1: unconnected-(J2-Pad1) -> /IOP/SDD2
- J5 pad 2: Net-(J2-Pad2) -> /IOP/SD~{CS}_D3
- J5 pad 3: Net-(J2-Pad3) -> /IOP/SDMOSI_CMD
- J5 pad 4: +3V3 -> SD3V3
- J5 pad 5: Net-(J2-Pad5) -> /IOP/SDSCK
- J5 pad 7: /MISOr -> /IOP/SDMISO_D0
- J5 pad 8: unconnected-(J2-Pad8) -> /IOP/SDD1
- J5 pad 9: /DETr -> /IOP/SD~{CD}
- R1 pad 1: /MOSI -> Net-(J4-Pin_9)
- R1 pad 2: Net-(J2-Pad3) -> GND
- R10 pad 1: Net-(Q4-Pad1) -> /IOP/Mac5Vsense
- R10 pad 2: /ESP32/IRQ -> GND
- R11 pad 1: /BusControl/ACK-2 -> /Control/~{PROG}
- R11 pad 2: /AddrLatch/ACLK -> /F~{PROG}
- R12 pad 1: /ESP32/TCK -> Net-(U16-CLK0)
- R12 pad 2: Net-(J4-Pad4) -> /Control/VGACLK
- R13 pad 1: +3V3 -> /Control/FTCKr
- R13 pad 2: /ESP32/IO0 -> /Control/FTCK
- R14 pad 1: /ESP32/TCK -> /FTCK
- R14 pad 2: GND -> /Control/FTCK
- R17 pad 1: /ESP32/IO2 -> (no net)
- R17 pad 2: GND -> (no net)
- R18 pad 1: +3V3 -> (no net)
- R18 pad 2: Net-(R18-Pad2) -> GND
- R19 pad 1: Net-(R18-Pad2) -> +3V3
- R19 pad 2: GND -> (no net)
- R2 pad 1: /S~{CS} -> Net-(U1E-PL35A)
- R2 pad 2: Net-(J2-Pad2) -> /Control/RCLK
- R20 pad 1: +3V3 -> (no net)
- R20 pad 2: /ESP32/TDO -> GND
- R3 pad 1: /SCK -> /Control/BCLK
- R3 pad 2: Net-(J2-Pad5) -> Net-(U5-4Y)
- R4 pad 1: /MISO -> /Control/B~{RES}
- R4 pad 2: /MISOr -> Net-(U18-4Y)
- R5 pad 1: /DET -> unconnected-(R5-Pad1)
- R5 pad 2: /DETr -> /Control/VSTRBi
- R6 pad 1: +3V3 -> Net-(U1C-~{PCK}20/PR23D)
- R6 pad 2: /MISOr -> /Control/VCLK
- R7 pad 1: +3V3 -> unconnected-(R7-Pad1)
- R7 pad 2: /DETr -> /Control/BV~{HSYNC}
- R8 pad 1: /BusControl/~{CLK}r -> unconnected-(R8-Pad1)
- R8 pad 2: /BusControl/~{CLK} -> /Control/BV~{VSYNC}
- R9 pad 1: Net-(R9-Pad1) -> Mac5V
- R9 pad 2: Net-(R9-Pad2) -> /IOP/Mac5Vsense
- U11 pad 1: /BusControl/REG~{OE} -> /Control/BID~{OE}
- U11 pad 10: GND -> /Control/BID~{OE}
- U11 pad 11: /CtrlStatReg/RDCLK -> /Control/B~{ID}_~{ARB}3
- U11 pad 12: /AddrLatch/~{AD}16 -> /NuBus/~{ID}3
- U11 pad 13: /AddrLatch/~{AD}17 -> /Control/BID~{OE}
- U11 pad 14: /AddrLatch/~{AD}18 -> +3V3
- U11 pad 2: /DataReg/RQ8 -> /NuBus/~{ID}0
- U11 pad 3: /DataReg/RQ9 -> /Control/B~{ID}_~{ARB}0
- U11 pad 4: /DataReg/RQ10 -> /Control/BID~{OE}
- U11 pad 5: /DataReg/RQ11 -> /NuBus/~{ID}1
- U11 pad 6: /DataReg/RQ12 -> /Control/B~{ID}_~{ARB}1
- U11 pad 7: /DataReg/RQ13 -> GND
- U11 pad 8: /DataReg/RQ14 -> /Control/B~{ID}_~{ARB}2
- U11 pad 9: /DataReg/RQ15 -> /NuBus/~{ID}2
- U12 pad 1: /BusControl/REG~{OE} -> /Control/OTM~{OE}
- U12 pad 10: GND -> /Control/BTM~{OE}
- U12 pad 11: /CtrlStatReg/RDCLK -> /Control/B~{TM}0
- U12 pad 12: /AddrLatch/~{AD}8 -> /NuBus/~{TM}0
- U12 pad 13: /AddrLatch/~{AD}9 -> /Control/BTM~{OE}
- U12 pad 14: /AddrLatch/~{AD}10 -> +3V3
- U12 pad 2: /DataReg/RQ16 -> /Control/B~{TM}0
- U12 pad 3: /DataReg/RQ17 -> /NuBus/~{TM}0
- U12 pad 4: /DataReg/RQ18 -> /Control/OTM~{OE}
- U12 pad 5: /DataReg/RQ19 -> /Control/B~{TM}1
- U12 pad 6: /DataReg/RQ20 -> /NuBus/~{TM}1
- U12 pad 7: /DataReg/RQ21 -> GND
- U12 pad 8: /DataReg/RQ22 -> /Control/B~{TM}1
- U12 pad 9: /DataReg/RQ23 -> /NuBus/~{TM}1
- U13 pad 1: /BusControl/REG~{OE} -> /Control/ARB~{OE}
- U13 pad 10: GND -> /Control/ARB~{OE}
- U13 pad 11: /CtrlStatReg/RDCLK -> /NuBus/~{ARB}1
- U13 pad 12: /AddrLatch/~{AD}0 -> /NuBus/~{ID}1
- U13 pad 13: /AddrLatch/~{AD}1 -> /Control/ARB~{OE}
- U13 pad 14: /AddrLatch/~{AD}2 -> +3V3
- U13 pad 2: /DataReg/RQ24 -> /NuBus/~{ID}2
- U13 pad 3: /DataReg/RQ25 -> /NuBus/~{ARB}2
- U13 pad 4: /DataReg/RQ26 -> /Control/ARB~{OE}
- U13 pad 5: /DataReg/RQ27 -> /NuBus/~{ID}3
- U13 pad 6: /DataReg/RQ28 -> /NuBus/~{ARB}3
- U13 pad 7: /DataReg/RQ29 -> GND
- U13 pad 8: /DataReg/RQ30 -> /NuBus/~{ARB}0
- U13 pad 9: /DataReg/RQ31 -> /NuBus/~{ID}0
- U14 pad 1: GND -> +3V3
- U14 pad 2: /AddrLatch/~{AD}5 -> GND
- U14 pad 3: /AddrLatch/~{AD}4 -> /IOP/SDPWR
- U14 pad 4: /AddrLatch/~{AD}3 -> unconnected-(U14-NC-Pad4)
- U14 pad 5: /AddrLatch/~{AD}2 -> SD3V3
- U14 pad 6: /AddrLatch/~{AD}1 -> SD3V3
- U15 pad 1: GND -> /D-
- U15 pad 2: /AddrLatch/~{AD}13 -> /D+
- U15 pad 3: /AddrLatch/~{AD}12 -> GND
- U16 pad 1: GND -> +3V3
- U16 pad 10: GND -> Net-(U16-CLK0)
- U16 pad 2: /AddrLatch/~{AD}21 -> Net-(U16-XA)
- U16 pad 3: /AddrLatch/~{AD}20 -> Net-(U16-XB)
- U16 pad 4: /AddrLatch/~{AD}19 -> /Control/SCL
- U16 pad 5: /AddrLatch/~{AD}18 -> /Control/SDA
- U16 pad 6: /AddrLatch/~{AD}17 -> unconnected-(U16-CLK2-Pad6)
- U16 pad 7: /AddrLatch/~{AD}16 -> +3V3
- U16 pad 8: /AddrLatch/~{AD}15 -> GND
- U16 pad 9: /AddrLatch/~{AD}14 -> unconnected-(U16-CLK1-Pad9)
- U17 pad 1: +3V3 -> /Control/OACK~{OE}
- U17 pad 10: +3V3 -> GND
- U17 pad 11: /BusControl/~{CLK} -> /Control/B~{ACK}
- U17 pad 12: /BusControl/~{ACK}-2 -> /NuBus/~{ACK}
- U17 pad 13: +3V3 -> GND
- U17 pad 2: /BusControl/~{CSTART} -> /Control/O~{ACK}
- U17 pad 3: /BusControl/~{CLK} -> /NuBus/~{ACK}
- U17 pad 4: +3V3 -> /Control/OSTART~{OE}
- U17 pad 5: /BusControl/~{ACK}-2 -> /Control/O~{START}
- U17 pad 6: /BusControl/ACK-2 -> /NuBus/~{START}
- U17 pad 8: /BusControl/ACK-1 -> /Control/B~{START}
- U17 pad 9: /BusControl/~{ACK}-1 -> /NuBus/~{START}
- U18 pad 1: +3V3 -> /IOP/ORES
- U18 pad 10: unconnected-(U18-Pad10) -> GND
- U18 pad 11: unconnected-(U18-Pad11) -> Net-(U18-4Y)
- U18 pad 12: unconnected-(U18-Pad12) -> /NuBus/~{RES}
- U18 pad 13: unconnected-(U18-Pad13) -> GND
- U18 pad 2: /BusControl/~{ACK}-1 -> GND
- U18 pad 3: /AddrLatch/~{AD}[31..0] -> /NuBus/~{RES}
- U18 pad 4: +3V3 -> GND
- U18 pad 5: /BusControl/~{ACK}-0 -> GND
- U18 pad 6: /BusControl/ACK-0 -> unconnected-(U18-2Y-Pad6)
- U18 pad 9: unconnected-(U18-Pad9) -> GND
- U2 pad 1: /AddrLatch/L~{A}21 -> GND
- U2 pad 10: /AddrLatch/L~{A}4 -> /Control/B~{RES}
- U2 pad 11: /AddrLatch/L~{A}3 -> /Control/EIRQ
- U2 pad 12: /AddrLatch/L~{A}2 -> /Control/DONE
- U2 pad 13: /ROM/RD0 -> /Control/QD3
- U2 pad 14: /ROM/RD1 -> /Control/Q~{CS}
- U2 pad 15: /ROM/RD2 -> /Control/DIN
- U2 pad 16: GND -> /Control/QSCK
- U2 pad 17: /ROM/RD3 -> /Control/DOUT
- U2 pad 18: /ROM/RD4 -> /Control/QD2
- U2 pad 19: /ROM/RD5 -> /Control/~{PROG}
- U2 pad 2: /AddrLatch/L~{A}18 -> GND
- U2 pad 20: /ROM/RD6 -> unconnected-(U2-IO16-Pad20)
- U2 pad 21: /ROM/RD7 -> /Control/CCLK
- U2 pad 22: GND -> /Control/CLK
- U2 pad 23: /AddrLatch/L~{A}12 -> /D-
- U2 pad 24: /BusControl/BDIR -> /D+
- U2 pad 25: /AddrLatch/L~{A}13 -> /IOP/SDPWR
- U2 pad 26: /AddrLatch/L~{A}11 -> /IOP/SD~{CD}
- U2 pad 27: /AddrLatch/L~{A}10 -> unconnected-(U2-NC-Pad27)
- U2 pad 28: /AddrLatch/L~{A}15 -> /IOP/SDD2
- U2 pad 29: /AddrLatch/L~{A}16 -> /IOP/SDD1
- U2 pad 3: /AddrLatch/L~{A}17 -> +3V3
- U2 pad 30: /AddrLatch/L~{A}20 -> GND
- U2 pad 31: /BusControl/ROM~{WE} -> /IOP/SDMISO_D0
- U2 pad 32: +5V -> /IOP/SDMOSI_CMD
- U2 pad 4: /AddrLatch/L~{A}14 -> /E~{DL}
- U2 pad 5: /AddrLatch/L~{A}9 -> /IOP/Mac5Vsense
- U2 pad 6: /AddrLatch/L~{A}8 -> /IOP/~{LED}
- U2 pad 7: /AddrLatch/L~{A}7 -> /IOP/ORES
- U2 pad 8: /AddrLatch/L~{A}6 -> /IOP/WarpEN
- U2 pad 9: /AddrLatch/L~{A}5 -> /IOP/B~{IPL}2
- U3 pad 1: GND -> +3V3
- U3 pad 10: unconnected-(U3-Pad10) -> /Control/RD5
- U3 pad 11: unconnected-(U3-Pad11) -> /Control/RD6
- U3 pad 12: unconnected-(U3-Pad12) -> GND
- U3 pad 13: /ESP32/DTR -> /Control/RD7
- U3 pad 14: /ESP32/RTS -> +3V3
- U3 pad 15: Net-(R18-Pad2) -> /Control/RDQML
- U3 pad 16: +3V3 -> /Control/R~{WE}
- U3 pad 2: /ESP32/DBG_RX -> /Control/RD0
- U3 pad 3: /ESP32/DBG_TX -> +3V3
- U3 pad 4: +3V3 -> /Control/RD1
- U3 pad 5: /ESP32/D+ -> /Control/RD2
- U3 pad 6: /ESP32/D- -> GND
- U3 pad 7: Net-(C1-Pad1) -> /Control/RD3
- U3 pad 8: Net-(C2-Pad1) -> /Control/RD4
- U3 pad 9: unconnected-(U3-Pad9) -> +3V3
- U4 pad 1: /BusControl/BDIR -> +3V3
- U4 pad 10: GND -> /Control/VD5
- U4 pad 11: /ROM/RD0 -> /Control/VD6
- U4 pad 12: /ROM/RD1 -> GND
- U4 pad 13: /ROM/RD2 -> /Control/VD7
- U4 pad 14: /ROM/RD3 -> +3V3
- U4 pad 15: /ROM/RD4 -> /Control/VDQML
- U4 pad 16: /ROM/RD5 -> /Control/V~{WE}
- U4 pad 17: /ROM/RD6 -> /Control/V~{CAS}
- U4 pad 18: /ROM/RD7 -> /Control/V~{RAS}
- U4 pad 19: /BusControl/~{ACK}-0 -> GND
- U4 pad 2: /AddrLatch/~{AD}31 -> /Control/VD0
- U4 pad 20: +3V3 -> /Control/VBA0
- U4 pad 3: /AddrLatch/~{AD}30 -> +3V3
- U4 pad 4: /AddrLatch/~{AD}29 -> /Control/VD1
- U4 pad 5: /AddrLatch/~{AD}28 -> /Control/VD2
- U4 pad 6: /AddrLatch/~{AD}27 -> GND
- U4 pad 7: /AddrLatch/~{AD}26 -> /Control/VD3
- U4 pad 8: /AddrLatch/~{AD}25 -> /Control/VD4
- U4 pad 9: /AddrLatch/~{AD}24 -> +3V3
- U5 pad 1: /DataReg/P~{OE} -> /Control/O~{NMRQ}
- U5 pad 11: /BusControl/REG~{WE} -> Net-(U5-4Y)
- U5 pad 12: /DataReg/Q33 -> /NuBus/CLK
- U5 pad 13: /DataReg/Q34 -> GND
- U5 pad 14: /DataReg/Q35 -> +3V3
- U5 pad 2: /AddrLatch/~{AD}31 -> GND
- U5 pad 3: /AddrLatch/~{AD}30 -> /NuBus/~{NMRQ}
- U5 pad 4: /AddrLatch/~{AD}29 -> /Control/O~{RQST}
- U5 pad 5: /AddrLatch/~{AD}28 -> GND
- U5 pad 6: /AddrLatch/~{AD}27 -> /NuBus/~{RQST}
- U5 pad 7: /AddrLatch/~{AD}26 -> GND
- U5 pad 8: /AddrLatch/~{AD}25 -> unconnected-(U5-3Y-Pad8)
- U5 pad 9: /AddrLatch/~{AD}24 -> GND
- U6 pad 1: /DataReg/P~{OE} -> /Control/BARB~{OE}
- U6 pad 10: GND -> /Control/BARB~{OE}
- U6 pad 11: /BusControl/REG~{WE} -> /Control/B~{ID}_~{ARB}1
- U6 pad 12: /DataReg/Q25 -> /NuBus/~{ARB}1
- U6 pad 13: /DataReg/Q26 -> /Control/BARB~{OE}
- U6 pad 14: /DataReg/Q27 -> +3V3
- U6 pad 2: /AddrLatch/~{AD}23 -> /NuBus/~{ARB}2
- U6 pad 3: /AddrLatch/~{AD}22 -> /Control/B~{ID}_~{ARB}2
- U6 pad 4: /AddrLatch/~{AD}21 -> /Control/BARB~{OE}
- U6 pad 5: /AddrLatch/~{AD}20 -> /NuBus/~{ARB}3
- U6 pad 6: /AddrLatch/~{AD}19 -> /Control/B~{ID}_~{ARB}3
- U6 pad 7: /AddrLatch/~{AD}18 -> GND
- U6 pad 8: /AddrLatch/~{AD}17 -> /Control/B~{ID}_~{ARB}0
- U6 pad 9: /AddrLatch/~{AD}16 -> /NuBus/~{ARB}0
Routing:
- net +3V3: track 2410.8 -> 160.5 mm, vias 314 -> 92
- net /BusControl/BDIR: track 331.2 -> 0.00 mm, vias 7 -> 0
- net /CtrlStatReg/~{RDREQ}: track 278.4 -> 0.00 mm, vias 5 -> 0
- net +5V: track 329.3 -> 52.2 mm, vias 11 -> 10
- net /BusControl/ROM~{WE}: track 266.5 -> 0.00 mm, vias 5 -> 0
- net /CtrlStatReg/~{WRREQ}: track 255.3 -> 0.00 mm, vias 4 -> 0
- net Net-(Q4-Pad1): track 248.5 -> 0.00 mm, vias 2 -> 0
- net /CtrlStatReg/RDCLK: track 225.9 -> 0.00 mm, vias 9 -> 0
- net /AddrLatch/L~{TM}1: track 210.0 -> 0.00 mm, vias 4 -> 0
- net /CtrlStatReg/WRCLK: track 208.8 -> 0.00 mm, vias 4 -> 0
- net /DataReg/P~{OE}: track 179.1 -> 0.00 mm, vias 10 -> 0
- net /CtrlStatReg/WR~{IE}: track 167.7 -> 0.00 mm, vias 4 -> 0
- net /DataReg/~{CS}: track 166.3 -> 0.00 mm, vias 7 -> 0
- net /CtrlStatReg/RD~{IE}: track 164.5 -> 0.00 mm, vias 4 -> 0
- net /ROM/RD7: track 161.5 -> 0.00 mm, vias 1 -> 0
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- added copper zone on B.Cu, net +3V3
- added copper zone on In3.Cu, net GND
- added copper zone on In4.Cu, net GND
Other:
- board size 193.7 x 101.6 mm -> 168.3 x 101.6 mm
- copper layers 4 -> 6
- rule pad_to_mask_clearance: 0 -> 0.0762
- board text added: "Video and I/O for Mac"
- board text added: "Videomatic"
- board text removed: "WiFi"
- board text removed: "for Macintosh"
