File: NuBus-ESP32.kicad_sch (KiCad schematic)
At the start: 21 parts, among them J2 Xunpu TF-115, J3 microUSB-B, U27 AZ1117EH-3.3TRG1

Commit message: idk
Parts:
- removed C4, C5: 10u, stdpads:C_0805, symbol Device:C_Small
- removed FID5: Fiducial, stdpads:Fiducial, symbol Mechanical:Fiducial
- removed J2: Xunpu TF-115, stdpads:Xunpu_TF-115_microSD, symbol GW_Connector:Micro_SD_SingleDet
- removed R2, R4, R5: 100, stdpads:R_0805, symbol Device:R_Small
- removed R3: 22, stdpads:R_0805, symbol Device:R_Small
- removed R6, R7: 47k, stdpads:R_0805, symbol Device:R_Small
- removed U27: AZ1117EH-3.3TRG1, stdpads:SOT-223, symbol GW_Power:AP1117-33
- added J2: UART, stdpads:Tag-Connect_TC2030-IDC-NL_2x03_P1.27mm_Vertical_with_bottom_clip, symbol Connector_Generic:Conn_02x03_Odd_Even
- added J4: EJTAG, stdpads:Tag-Connect_TC2050-IDC-NL_2x05_P1.27mm_Vertical_with_bottom_clip, symbol Connector_Generic:Conn_02x05_Odd_Even
- added J5: microSD, stdpads:Xunpu_TF-115_microSD, symbol Connector:Micro_SD_Card_Det1
- added J6: FJTAG, stdpads:Tag-Connect_TC2050-IDC-NL_2x05_P1.27mm_Vertical_with_bottom_clip, symbol Connector_Generic:Conn_02x05_Odd_Even
- added J7: VGA, symbol Connector:DE15_Plug_HighDensity_MountingHoles
- added R11, R14: 68, stdpads:R_0603, symbol Device:R_Small
- added SW1: DL, symbol Switch:SW_Push
- added U15: TPD2EUSB30, stdpads:TI_DRT-3, symbol Power_Protection:TPD2EUSB30
- H1, H2, H3, H4: value (none) -> ~
- J3: value microUSB-B -> microUSB; footprint stdpads:USB_Micro-B_ShouHan_MicroXNJ -> stdpads:USB_Micro-B_Amphenol_10118192-0001; LCSC Part C404969 -> (none)
- R1: value 100 -> 33; footprint stdpads:R_0805 -> stdpads:R_0603; LCSC Part C17408 -> (none)
Connections:
- net +3V3: now also J2.2 (Pin_2), J4.1 (Pin_1), J6.6 (Pin_6)
- net GND: now also R1.2, J2.4 (Pin_4), J4.3 (Pin_3), J4.5 (Pin_5), J4.7 (Pin_7), J5.10 (SHIELD), J5.6 (VSS), J6.2 (Pin_2), J6.4 (Pin_4), J6.8 (Pin_8), J7.0, J7.10, J7.5, J7.6, J7.7, J7.8, SW1.2, U15.3 (GND)
- net USB5V: now reaches J3.1 (VBUS)
- net ESP32/D+ renamed D+
- net D+: now also U15.2 (D-)
- net ESP32/D- renamed D-
- net D-: now also U15.1 (D+)
- net MOSI: no longer names the net of R1.1
- net MOSI: now also J4.9 (Pin_9)
- new net Control/FTCK: R14.2
- new net Control/~{PROG}: R11.1
- new net ERX: J2.3 (Pin_3)
- new net ETCK: J4.4 (Pin_4)
- new net ETDI: J4.8 (Pin_8)
- new net ETDO: J4.6 (Pin_6)
- new net ETMS: J4.2 (Pin_2)
- new net ETX: J2.1 (Pin_1)
- new net E~{DL}: J2.6 (Pin_6), SW1.1
- new net E~{RES}: J2.5 (Pin_5), J4.10 (Pin_10)
- new net FTCK: J6.1 (Pin_1), R14.1
- new net FTDI: J6.5 (Pin_5)
- new net FTDO: J6.7 (Pin_7)
- new net FTMS: J6.3 (Pin_3)
- new net F~{PROG}: J6.10 (Pin_10), R11.2
- new net IOP/SDD1: J5.8 (DAT1)
- new net IOP/SDD2: J5.1 (DAT2)
- new net IOP/SDMISO_D0: J5.7 (DAT0)
- new net IOP/SDMOSI_CMD: J5.3 (CMD)
- new net IOP/SDSCK: J5.5 (CLK)
- new net IOP/SD~{CD}: J5.9 (DET)
- new net IOP/SD~{CS}_D3: J5.2 (DAT3/CD)
- new net SD3V3: J5.4 (VDD)
- new net VB: J7.3
- new net VG: J7.2
- new net VR: J7.1
- new net V~{HSYNC}: J7.13
- new net V~{VSYNC}: J7.14
- no-connect marks 3 -> 2
Other:
- removed sheet AddrLatch
- removed sheet BusControl
- removed sheet CtrlStatReg
- removed sheet DataReg
- removed sheet ESP32
- removed sheet ROM
- added sheet Control (Control.kicad_sch)
- added sheet IOP (IOP.kicad_sch)
- added sheet NuBusBuf (NuBusBuf.kicad_sch)
- added sheet Power (Power.kicad_sch)
- added sheet RAM (RAM.kicad_sch)
- added sheet VCLK (VCLK.kicad_sch)
- added sheet VDAC (VDAC.kicad_sch)
- added sheet VRAM (VRAM.kicad_sch)
- sheet NuBus ports: added ~{ARB}[3..0], ~{PFW}, ~{RQST}; removed none
- moved on the sheet: FID1, FID2, FID3, FID4, H1, H2, H3, H4
