File: NuBus.kicad_sch (KiCad schematic)
At the start: 3 parts, among them J1 MacNuBus

Commit message: work on FPGA
Parts:
- added C? (x4): 10u, stdpads:C_0805, symbol Device:C_Small
Connections:
- net +5V: now also C?.1, C?.1
- net GND: now also C?.1, C?.2, C?.2, C?.2
- net -12V: now reaches J1.A1 (-12V)
- net -12V: now also J1.B1 (-12V), C?.2
- net +12V: now reaches J1.A32 (+12V)
- net +12V: now also J1.B32 (+12V), C?.1
- no-connect marks 22 -> 18
Other:
- moved on the sheet: C34, C35

Commit message: Revert "work on FPGA"
This reverts commit a96523e8d17974c7c48efc8a38ae046f7948cd49.
Parts:
- removed C? (x4): 10u, stdpads:C_0805, symbol Device:C_Small
Connections:
- net +12V: no longer names the net of J1.A32 (+12V)
- net +12V: no longer J1.B32 (+12V)
- net -12V: no longer names the net of J1.A1 (-12V)
- net -12V: no longer J1.B1 (-12V)
- no-connect marks 18 -> 22
Other:
- moved on the sheet: C34, C35

Commit message: idk
Connections:
- net ~{ARB}1: now reaches J1.A24 (~{ARB}1)
- net ~{ARB}3: now reaches J1.A25 (~{ARB}3)
- net ~{RQST}: now reaches J1.A30 (~{RQST})
- net ~{PFW}: now reaches J1.C23 (~{PFW})
- net ~{ARB}0: now reaches J1.C24 (~{ARB}0)
- net ~{ARB}2: now reaches J1.C25 (~{ARB}2)
- no-connect marks 22 -> 16
